File: Electronics/PiKwonDoHAT/PiKwonDoHAT.sch (KiCad schematic (older format))
At the start: 42 parts, among them J1 Conn_02x20_Odd_Even, J2 Judge3, J3 Judge2, J4 Judge1, J5 Controller, U1 74LV1T34, U2 74LV1T34, U3 74LV1T34, U4 74LV1T34

Commit message: Tweaked schematic a bit further; changed PCB references to match schematic.
Parts:
- CN2: renamed from J2; value Judge3 -> Judge1
- CN4: renamed from J4; value Judge1 -> Judge3
- renumbered J3 to CN3, J5 to CN5
Connections:
- net labels removed: C_Data, J1_Data, J2_Data, J3_Data
Changed lines of the file:
@@
 Sheet 1 1
 Title ""
-Date ""
+Date "2018-7-28.1"
 Rev ""
 Comp ""
@@
 $EndDescr
 $Comp
-L RJ12-UNSHLD J2
+L RJ12-UNSHLD CN2
 U 1 1 5B25A715
 P 9300 1600
-F 0 "J2" H 9500 2100 50  0000 C CNN
-F 1 "Judge3" H 9150 2100 50  0000 C CNN
+F 0 "CN2" H 9500 2100 50  0000 C CNN
+F 1 "Judge1" H 9150 2100 50  0000 C CNN
 F 2 "PiKwonDo:TH-RJ12" H 9300 1600 50  0001 C CNN
 F 3 "" H 9300 1600 50  0001 C CNN
@@
 $EndComp
 $Comp
-L RJ12-UNSHLD J3
+L RJ12-UNSHLD CN3
 U 1 1 5B25A769
 P 9300 2900
-F 0 "J3" H 9500 3400 50  0000 C CNN
+F 0 "CN3" H 9500 3400 50  0000 C CNN
 F 1 "Judge2" H 9150 3400 50  0000 C CNN
 F 2 "PiKwonDo:TH-RJ12" H 9300 2900 50  0001 C CNN
@@
 $EndComp
 $Comp
-L RJ12-UNSHLD J4
+L RJ12-UNSHLD CN4
 U 1 1 5B25A78D
 P 9300 4200
-F 0 "J4" H 9500 4700 50  0000 C CNN
-F 1 "Judge1" H 9150 4700 50  0000 C CNN
+F 0 "CN4" H 9500 4700 50  0000 C CNN
+F 1 "Judge3" H 9150 4700 50  0000 C CNN
 F 2 "PiKwonDo:TH-RJ12" H 9300 4200 50  0001 C CNN
 F 3 "" H 9300 4200 50  0001 C CNN
@@
 $EndComp
 $Comp
-L RJ12-UNSHLD J5
+L RJ12-UNSHLD CN5
 U 1 1 5B25A7B5
 P 9300 5500
-F 0 "J5" H 9500 6000 50  0000 C CNN
+F 0 "CN5" H 9500 6000 50  0000 C CNN
 F 1 "Controller" H 9150 6000 50  0000 C CNN
 F 2 "PiKwonDo:TH-RJ12" H 9300 5500 50  0001 C CNN
@@
 	3000 2900 2600 2900
 Text Label 2600 3000 0    60   ~ 0
-J1_Data
+J1_DATA
 Text Label 2600 2900 0    60   ~ 0
 J1_LOAD
@@
 	3000 3300 2600 3300
 Text Label 2600 3400 0    60   ~ 0
-J2_Data
+J2_DATA
 Text Label 2600 3300 0    60   ~ 0
 J2_LOAD
@@
 	3000 3700 2600 3700
 Text Label 2600 3800 0    60   ~ 0
-J3_Data
+J3_DATA
 Text Label 2600 3700 0    60   ~ 0
 J3_LOAD
@@
 	3000 4400 2600 4400
 Text Label 2600 4500 0    60   ~ 0
-C_Data
+C_DATA
 Text Label 2600 4400 0    60   ~ 0
 C_LOAD

Commit message: Synchronized PCB with schematic netlist.
Parts:
- renumbered J1 to CN1
Changed lines of the file:
@@
 $EndComp
 $Comp
-L Conn_02x20_Odd_Even J1
+L Conn_02x20_Odd_Even CN1
 U 1 1 5B25D769
 P 3300 3700
-F 0 "J1" H 3350 4700 50  0000 C CNN
+F 0 "CN1" H 3350 4700 50  0000 C CNN
 F 1 "Conn_02x20_Odd_Even" H 3350 2600 50  0000 C CNN
 F 2 "Pin_Headers:Pin_Header_Straight_2x20_Pitch2.54mm" H 3300 3700 50  0001 C CNN

Commit message: Changed diode footprints to SOD-323 (Hand)
Parts:
- D1, D2, D3, D4, D5, D6, D7, D8, D9: footprint Diodes_SMD:SOD-80C -> Diodes_SMD:D_SOD-323_HandSoldering
