File: Electronics/PiKwonDoHAT/PiKwonDoHAT.sch (KiCad schematic (older format))
At the start: 42 parts, among them CN1 Conn_02x20_Odd_Even, CN2 Judge1, CN3 Judge2, CN4 Judge3, CN5 Controller, U1 74LV1T34, U2 74LV1T34, U3 74LV1T34, U4 74LV1T34

Commit message: Trace widening for manufacturing and assembly ese
Parts:
- CN1: symbol Conn_02x20_Odd_Even -> Connector_Generic_MountingPin:Conn_02x20_Odd_Even_MountingPin
- CN2, CN3, CN4, CN5: symbol RJ12-UNSHLD -> PiKwonDo:RJ12-UNSHLD
- U1, U2, U3, U4: symbol 74LV1T34 -> PiKwonDo:SN74LV1T34DBVR
Connections:
- wire segments 91 -> 93
Other:
- moved on the sheet: C1, C2, C3, C4

Commit message: Updated HAT trace widths
Connections:
- no-connect marks 31 -> 32
Changed lines of the file:
@@
 Wire Wire Line
 	6050 1350 5900 1350
+NoConn ~ 3250 2500
 $EndSCHEMATC

Commit message: Updated library footprint references
Parts:
- C1, C2, C3, C4: footprint Capacitors_SMD:C_0805_HandSoldering -> Capacitor_SMD:C_0805_2012Metric_Pad1.15x1.40mm_HandSolder
- C10, C11, C12, C5, C6, C7, C8, C9: footprint Capacitors_SMD:C_0603_HandSoldering -> Capacitor_SMD:C_0805_2012Metric_Pad1.15x1.40mm_HandSolder
- CN1: footprint Pin_Headers:Pin_Header_Straight_2x20_Pitch2.54mm -> Connector_PinSocket_2.54mm:PinSocket_2x20_P2.54mm_Vertical
Connections:
- no-connect marks 32 -> 31
Changed lines of the file:
@@
 F 0 "CN1" H 3350 4700 50  0000 C CNN
 F 1 "Conn_02x20_Odd_Even" H 3350 2600 50  0000 C CNN
-F 2 "Pin_Headers:Pin_Header_Straight_2x20_Pitch2.54mm" H 3300 3700 50  0001 C CNN
+F 2 "Connector_PinSocket_2.54mm:PinSocket_2x20_P2.54mm_Vertical" H 3300 3700 50  0001 C CNN
 F 3 "" H 3300 3700 50  0001 C CNN
 	1    3300 3700
@@
 F 0 "C6" H 8375 2000 50  0000 L CNN
 F 1 "470pF" H 8375 1800 50  0000 L CNN
-F 2 "Capacitors_SMD:C_0603_HandSoldering" H 8388 1750 50  0001 C CNN
+F 2 "Capacitor_SMD:C_0805_2012Metric_Pad1.15x1.40mm_HandSolder" H 8388 1750 50  0001 C CNN
 F 3 "" H 8350 1900 50  0001 C CNN
 	1    8350 1900
@@
 F 0 "C5" H 8025 2000 50  0000 L CNN
 F 1 "470pF" H 8025 1800 50  0000 L CNN
-F 2 "Capacitors_SMD:C_0603_HandSoldering" H 8038 1750 50  0001 C CNN
+F 2 "Capacitor_SMD:C_0805_2012Metric_Pad1.15x1.40mm_HandSolder" H 8038 1750 50  0001 C CNN
 F 3 "" H 8000 1900 50  0001 C CNN
 	1    8000 1900
@@
 F 0 "C8" H 8375 3300 50  0000 L CNN
 F 1 "470pF" H 8375 3100 50  0000 L CNN
-F 2 "Capacitors_SMD:C_0603_HandSoldering" H 8388 3050 50  0001 C CNN
+F 2 "Capacitor_SMD:C_0805_2012Metric_Pad1.15x1.40mm_HandSolder" H 8388 3050 50  0001 C CNN
 F 3 "" H 8350 3200 50  0001 C CNN
 	1    8350 3200
@@
 F 0 "C7" H 8025 3300 50  0000 L CNN
 F 1 "470pF" H 8025 3100 50  0000 L CNN
-F 2 "Capacitors_SMD:C_0603_HandSoldering" H 8038 3050 50  0001 C CNN
+F 2 "Capacitor_SMD:C_0805_2012Metric_Pad1.15x1.40mm_HandSolder" H 8038 3050 50  0001 C CNN
 F 3 "" H 8000 3200 50  0001 C CNN
 	1    8000 3200
@@
 F 0 "C10" H 8375 4600 50  0000 L CNN
 F 1 "470pF" H 8375 4400 50  0000 L CNN
-F 2 "Capacitors_SMD:C_0603_HandSoldering" H 8388 4350 50  0001 C CNN
+F 2 "Capacitor_SMD:C_0805_2012Metric_Pad1.15x1.40mm_HandSolder" H 8388 4350 50  0001 C CNN
 F 3 "" H 8350 4500 50  0001 C CNN
 	1    8350 4500
@@
 F 0 "C9" H 8025 4600 50  0000 L CNN
 F 1 "470pF" H 8025 4400 50  0000 L CNN
-F 2 "Capacitors_SMD:C_0603_HandSoldering" H 8038 4350 50  0001 C CNN
+F 2 "Capacitor_SMD:C_0805_2012Metric_Pad1.15x1.40mm_HandSolder" H 8038 4350 50  0001 C CNN
 F 3 "" H 8000 4500 50  0001 C CNN
 	1    8000 4500
@@
 F 0 "C12" H 8375 5900 50  0000 L CNN
 F 1 "470pF" H 8375 5700 50  0000 L CNN
-F 2 "Capacitors_SMD:C_0603_HandSoldering" H 8388 5650 50  0001 C CNN
+F 2 "Capacitor_SMD:C_0805_2012Metric_Pad1.15x1.40mm_HandSolder" H 8388 5650 50  0001 C CNN
 F 3 "" H 8350 5800 50  0001 C CNN
 	1    8350 5800
@@
 F 0 "C11" H 8025 5900 50  0000 L CNN
 F 1 "470pF" H 8025 5700 50  0000 L CNN
-F 2 "Capacitors_SMD:C_0603_HandSoldering" H 8038 5650 50  0001 C CNN
+F 2 "Capacitor_SMD:C_0805_2012Metric_Pad1.15x1.40mm_HandSolder" H 8038 5650 50  0001 C CNN
 F 3 "" H 8000 5800 50  0001 C CNN
 	1    8000 5800
@@
 F 0 "C2" V 4950 2400 50  0000 C CNN
 F 1 "10nF" V 5025 2475 50  0000 L CNN
-F 2 "Capacitors_SMD:C_0805_HandSoldering" H 5138 2250 50  0001 C CNN
+F 2 "Capacitor_SMD:C_0805_2012Metric_Pad1.15x1.40mm_HandSolder" H 5138 2250 50  0001 C CNN
 F 3 "" H 5100 2400 50  0001 C CNN
 	1    5100 2400
@@
 F 0 "C1" V 4950 950 50  0000 C CNN
 F 1 "10nF" V 5025 1025 50  0000 L CNN
-F 2 "Capacitors_SMD:C_0805_HandSoldering" H 5138 800 50  0001 C CNN
+F 2 "Capacitor_SMD:C_0805_2012Metric_Pad1.15x1.40mm_HandSolder" H 5138 800 50  0001 C CNN
 F 3 "" H 5100 950 50  0001 C CNN
 	1    5100 950
@@
 F 0 "C4" V 4950 5000 50  0000 C CNN
 F 1 "10nF" V 5025 5075 50  0000 L CNN
-F 2 "Capacitors_SMD:C_0805_HandSoldering" H 5138 4850 50  0001 C CNN
+F 2 "Capacitor_SMD:C_0805_2012Metric_Pad1.15x1.40mm_HandSolder" H 5138 4850 50  0001 C CNN
 F 3 "" H 5100 5000 50  0001 C CNN
 	1    5100 5000
@@
 F 0 "C3" V 4950 3700 50  0000 C CNN
 F 1 "10nF" V 5025 3775 50  0000 L CNN
-F 2 "Capacitors_SMD:C_0805_HandSoldering" H 5138 3550 50  0001 C CNN
+F 2 "Capacitor_SMD:C_0805_2012Metric_Pad1.15x1.40mm_HandSolder" H 5138 3550 50  0001 C CNN
 F 3 "" H 5100 3700 50  0001 C CNN
 	1    5100 3700
@@
 Wire Wire Line
 	6050 1350 5900 1350
-NoConn ~ 3250 2500
 $EndSCHEMATC

Commit message: Updated zener diode footprint and layout
Parts:
- C1, C10, C11, C12, C2, C3, C4, C5, C6, C7, C8, C9: footprint Capacitor_SMD:C_0805_2012Metric_Pad1.15x1.40mm_HandSolder -> Capacitor_SMD:C_1206_3216Metric_Pad1.42x1.75mm_HandSolder
- D2, D3, D4, D5, D6, D7, D8, D9: footprint Diodes_SMD:D_SOD-323_HandSoldering -> Diode_SMD:D_SOD-123
Changed lines of the file:
@@
 F 0 "D2" V 6650 1925 50  0000 L CNN
 F 1 "3.3V" V 6850 1925 50  0000 L CNN
-F 2 "Diodes_SMD:D_SOD-323_HandSoldering" H 6750 1900 50  0001 C CNN
+F 2 "Diode_SMD:D_SOD-123" H 6750 1900 50  0001 C CNN
 F 3 "" H 6750 1900 50  0001 C CNN
 	1    6750 1900
@@
 F 0 "D3" V 7000 1925 50  0000 L CNN
 F 1 "3.3V" V 7200 1925 50  0000 L CNN
-F 2 "Diodes_SMD:D_SOD-323_HandSoldering" H 7100 1900 50  0001 C CNN
+F 2 "Diode_SMD:D_SOD-123" H 7100 1900 50  0001 C CNN
 F 3 "" H 7100 1900 50  0001 C CNN
 	1    7100 1900
@@
 F 0 "C6" H 8375 2000 50  0000 L CNN
 F 1 "470pF" H 8375 1800 50  0000 L CNN
-F 2 "Capacitor_SMD:C_0805_2012Metric_Pad1.15x1.40mm_HandSolder" H 8388 1750 50  0001 C CNN
+F 2 "Capacitor_SMD:C_1206_3216Metric_Pad1.42x1.75mm_HandSolder" H 8388 1750 50  0001 C CNN
 F 3 "" H 8350 1900 50  0001 C CNN
 	1    8350 1900
@@
 F 0 "C5" H 8025 2000 50  0000 L CNN
 F 1 "470pF" H 8025 1800 50  0000 L CNN
-F 2 "Capacitor_SMD:C_0805_2012Metric_Pad1.15x1.40mm_HandSolder" H 8038 1750 50  0001 C CNN
+F 2 "Capacitor_SMD:C_1206_3216Metric_Pad1.42x1.75mm_HandSolder" H 8038 1750 50  0001 C CNN
 F 3 "" H 8000 1900 50  0001 C CNN
 	1    8000 1900
@@
 F 0 "C8" H 8375 3300 50  0000 L CNN
 F 1 "470pF" H 8375 3100 50  0000 L CNN
-F 2 "Capacitor_SMD:C_0805_2012Metric_Pad1.15x1.40mm_HandSolder" H 8388 3050 50  0001 C CNN
+F 2 "Capacitor_SMD:C_1206_3216Metric_Pad1.42x1.75mm_HandSolder" H 8388 3050 50  0001 C CNN
 F 3 "" H 8350 3200 50  0001 C CNN
 	1    8350 3200
@@
 F 0 "C7" H 8025 3300 50  0000 L CNN
 F 1 "470pF" H 8025 3100 50  0000 L CNN
-F 2 "Capacitor_SMD:C_0805_2012Metric_Pad1.15x1.40mm_HandSolder" H 8038 3050 50  0001 C CNN
+F 2 "Capacitor_SMD:C_1206_3216Metric_Pad1.42x1.75mm_HandSolder" H 8038 3050 50  0001 C CNN
 F 3 "" H 8000 3200 50  0001 C CNN
 	1    8000 3200
@@
 F 0 "C10" H 8375 4600 50  0000 L CNN
 F 1 "470pF" H 8375 4400 50  0000 L CNN
-F 2 "Capacitor_SMD:C_0805_2012Metric_Pad1.15x1.40mm_HandSolder" H 8388 4350 50  0001 C CNN
+F 2 "Capacitor_SMD:C_1206_3216Metric_Pad1.42x1.75mm_HandSolder" H 8388 4350 50  0001 C CNN
 F 3 "" H 8350 4500 50  0001 C CNN
 	1    8350 4500
@@
 F 0 "C9" H 8025 4600 50  0000 L CNN
 F 1 "470pF" H 8025 4400 50  0000 L CNN
-F 2 "Capacitor_SMD:C_0805_2012Metric_Pad1.15x1.40mm_HandSolder" H 8038 4350 50  0001 C CNN
+F 2 "Capacitor_SMD:C_1206_3216Metric_Pad1.42x1.75mm_HandSolder" H 8038 4350 50  0001 C CNN
 F 3 "" H 8000 4500 50  0001 C CNN
 	1    8000 4500
@@
 F 0 "C12" H 8375 5900 50  0000 L CNN
 F 1 "470pF" H 8375 5700 50  0000 L CNN
-F 2 "Capacitor_SMD:C_0805_2012Metric_Pad1.15x1.40mm_HandSolder" H 8388 5650 50  0001 C CNN
+F 2 "Capacitor_SMD:C_1206_3216Metric_Pad1.42x1.75mm_HandSolder" H 8388 5650 50  0001 C CNN
 F 3 "" H 8350 5800 50  0001 C CNN
 	1    8350 5800
@@
 F 0 "C11" H 8025 5900 50  0000 L CNN
 F 1 "470pF" H 8025 5700 50  0000 L CNN
-F 2 "Capacitor_SMD:C_0805_2012Metric_Pad1.15x1.40mm_HandSolder" H 8038 5650 50  0001 C CNN
+F 2 "Capacitor_SMD:C_1206_3216Metric_Pad1.42x1.75mm_HandSolder" H 8038 5650 50  0001 C CNN
 F 3 "" H 8000 5800 50  0001 C CNN
 	1    8000 5800
@@
 F 0 "C2" V 4950 2400 50  0000 C CNN
 F 1 "10nF" V 5025 2475 50  0000 L CNN
-F 2 "Capacitor_SMD:C_0805_2012Metric_Pad1.15x1.40mm_HandSolder" H 5138 2250 50  0001 C CNN
+F 2 "Capacitor_SMD:C_1206_3216Metric_Pad1.42x1.75mm_HandSolder" H 5138 2250 50  0001 C CNN
 F 3 "" H 5100 2400 50  0001 C CNN
 	1    5100 2400
@@
 F 0 "D4" V 6650 3225 50  0000 L CNN
 F 1 "3.3V" V 6850 3225 50  0000 L CNN
-F 2 "Diodes_SMD:D_SOD-323_HandSoldering" H 6750 3200 50  0001 C CNN
+F 2 "Diode_SMD:D_SOD-123" H 6750 3200 50  0001 C CNN
 F 3 "" H 6750 3200 50  0001 C CNN
 	1    6750 3200
@@
 F 0 "D5" V 7000 3225 50  0000 L CNN
 F 1 "3.3V" V 7200 3225 50  0000 L CNN
-F 2 "Diodes_SMD:D_SOD-323_HandSoldering" H 7100 3200 50  0001 C CNN
+F 2 "Diode_SMD:D_SOD-123" H 7100 3200 50  0001 C CNN
 F 3 "" H 7100 3200 50  0001 C CNN
 	1    7100 3200
@@
 F 0 "D6" V 6650 4525 50  0000 L CNN
 F 1 "3.3V" V 6850 4525 50  0000 L CNN
-F 2 "Diodes_SMD:D_SOD-323_HandSoldering" H 6750 4500 50  0001 C CNN
+F 2 "Diode_SMD:D_SOD-123" H 6750 4500 50  0001 C CNN
 F 3 "" H 6750 4500 50  0001 C CNN
 	1    6750 4500
@@
 F 0 "D7" V 7000 4525 50  0000 L CNN
 F 1 "3.3V" V 7200 4525 50  0000 L CNN
-F 2 "Diodes_SMD:D_SOD-323_HandSoldering" H 7100 4500 50  0001 C CNN
+F 2 "Diode_SMD:D_SOD-123" H 7100 4500 50  0001 C CNN
 F 3 "" H 7100 4500 50  0001 C CNN
 	1    7100 4500
@@
 F 0 "D8" V 6650 5825 50  0000 L CNN
 F 1 "3.3V" V 6850 5825 50  0000 L CNN
-F 2 "Diodes_SMD:D_SOD-323_HandSoldering" H 6750 5800 50  0001 C CNN
+F 2 "Diode_SMD:D_SOD-123" H 6750 5800 50  0001 C CNN
 F 3 "" H 6750 5800 50  0001 C CNN
 	1    6750 5800
@@
 F 0 "D9" V 7000 5825 50  0000 L CNN
 F 1 "3.3V" V 7200 5825 50  0000 L CNN
-F 2 "Diodes_SMD:D_SOD-323_HandSoldering" H 7100 5800 50  0001 C CNN
+F 2 "Diode_SMD:D_SOD-123" H 7100 5800 50  0001 C CNN
 F 3 "" H 7100 5800 50  0001 C CNN
 	1    7100 5800
@@
 F 0 "C1" V 4950 950 50  0000 C CNN
 F 1 "10nF" V 5025 1025 50  0000 L CNN
-F 2 "Capacitor_SMD:C_0805_2012Metric_Pad1.15x1.40mm_HandSolder" H 5138 800 50  0001 C CNN
+F 2 "Capacitor_SMD:C_1206_3216Metric_Pad1.42x1.75mm_HandSolder" H 5138 800 50  0001 C CNN
 F 3 "" H 5100 950 50  0001 C CNN
 	1    5100 950
@@
 F 0 "C4" V 4950 5000 50  0000 C CNN
 F 1 "10nF" V 5025 5075 50  0000 L CNN
-F 2 "Capacitor_SMD:C_0805_2012Metric_Pad1.15x1.40mm_HandSolder" H 5138 4850 50  0001 C CNN
+F 2 "Capacitor_SMD:C_1206_3216Metric_Pad1.42x1.75mm_HandSolder" H 5138 4850 50  0001 C CNN
 F 3 "" H 5100 5000 50  0001 C CNN
 	1    5100 5000
@@
 F 0 "C3" V 4950 3700 50  0000 C CNN
 F 1 "10nF" V 5025 3775 50  0000 L CNN
-F 2 "Capacitor_SMD:C_0805_2012Metric_Pad1.15x1.40mm_HandSolder" H 5138 3550 50  0001 C CNN
+F 2 "Capacitor_SMD:C_1206_3216Metric_Pad1.42x1.75mm_HandSolder" H 5138 3550 50  0001 C CNN
 F 3 "" H 5100 3700 50  0001 C CNN
 	1    5100 3700

Commit message: Updated trace routing and RJ12 footprint.
Parts:
- removed CN1: Conn_02x20_Odd_Even, Connector_PinSocket_2.54mm:PinSocket_2x20_P2.54mm_Vertical, symbol Connector_Generic_MountingPin:Conn_02x20_Odd_Even_MountingPin
- removed CN2: Judge1, PiKwonDo:TH-RJ12, symbol PiKwonDo:RJ12-UNSHLD
- removed CN3: Judge2, PiKwonDo:TH-RJ12, symbol PiKwonDo:RJ12-UNSHLD
- removed CN4: Judge3, PiKwonDo:TH-RJ12, symbol PiKwonDo:RJ12-UNSHLD
- removed CN5: Controller, PiKwonDo:TH-RJ12, symbol PiKwonDo:RJ12-UNSHLD
- added J1, J2, J3, J4: RJ10, Local_lib:RJ14, symbol Connector:RJ10
- added J5: Conn_02x20_Odd_Even, Connector_PinSocket_2.54mm:PinSocket_2x20_P2.54mm_Vertical, symbol Connector_Generic:Conn_02x20_Odd_Even
Connections:
- no-connect marks 31 -> 23
Changed lines of the file:
@@
 $EndDescr
-$Comp
-L PiKwonDo:RJ12-UNSHLD CN2
-U 1 1 5B25A715
-P 9300 1600
-F 0 "CN2" H 9500 2100 50  0000 C CNN
-F 1 "Judge1" H 9150 2100 50  0000 C CNN
-F 2 "PiKwonDo:TH-RJ12" H 9300 1600 50  0001 C CNN
-F 3 "" H 9300 1600 50  0001 C CNN
-	1    9300 1600
-	0    1    1    0
-$EndComp
-$Comp
-L PiKwonDo:RJ12-UNSHLD CN3
-U 1 1 5B25A769
-P 9300 2900
-F 0 "CN3" H 9500 3400 50  0000 C CNN
-F 1 "Judge2" H 9150 3400 50  0000 C CNN
-F 2 "PiKwonDo:TH-RJ12" H 9300 2900 50  0001 C CNN
-F 3 "" H 9300 2900 50  0001 C CNN
-	1    9300 2900
-	0    1    1    0
-$EndComp
-$Comp
-L PiKwonDo:RJ12-UNSHLD CN4
-U 1 1 5B25A78D
-P 9300 4200
-F 0 "CN4" H 9500 4700 50  0000 C CNN
-F 1 "Judge3" H 9150 4700 50  0000 C CNN
-F 2 "PiKwonDo:TH-RJ12" H 9300 4200 50  0001 C CNN
-F 3 "" H 9300 4200 50  0001 C CNN
-	1    9300 4200
-	0    1    1    0
-$EndComp
-$Comp
-L PiKwonDo:RJ12-UNSHLD CN5
-U 1 1 5B25A7B5
-P 9300 5500
-F 0 "CN5" H 9500 6000 50  0000 C CNN
-F 1 "Controller" H 9150 6000 50  0000 C CNN
-F 2 "PiKwonDo:TH-RJ12" H 9300 5500 50  0001 C CNN
-F 3 "" H 9300 5500 50  0001 C CNN
-	1    9300 5500
-	0    1    1    0
-$EndComp
 $Comp
 L power:PWR_FLAG #FLG01
@@
 $EndComp
 $Comp
-L Connector_Generic_MountingPin:Conn_02x20_Odd_Even_MountingPin CN1
-U 1 1 5B25D769
-P 3300 3700
-F 0 "CN1" H 3350 4700 50  0000 C CNN
-F 1 "Conn_02x20_Odd_Even" H 3350 2600 50  0000 C CNN
-F 2 "Connector_PinSocket_2.54mm:PinSocket_2x20_P2.54mm_Vertical" H 3300 3700 50  0001 C CNN
-F 3 "" H 3300 3700 50  0001 C CNN
-	1    3300 3700
-	-1   0    0    1
-$EndComp
-$Comp
 L power:GND #PWR03
 U 1 1 5B2ADD76
@@
 	0    1    1    0
 $EndComp
-NoConn ~ 8850 1400
-NoConn ~ 8850 1900
-NoConn ~ 8850 2700
-NoConn ~ 8850 3200
-NoConn ~ 8850 4000
-NoConn ~ 8850 4500
-NoConn ~ 8850 5300
-NoConn ~ 8850 5800
 Text Label 4900 2800 0    60   ~ 0
 J2_CLK
@@
 Wire Wire Line
 	6050 1350 5900 1350
+$Comp
+L Connector:RJ10 J1
+U 1 1 5C3E11E7
+P 9250 1700
+F 0 "J1" H 8920 1796 50  0000 R CNN
+F 1 "RJ10" H 8920 1705 50  0000 R CNN
+F 2 "Local_lib:RJ14" V 9250 1750 50  0001 C CNN
+F 3 "~" V 9250 1750 50  0001 C CNN
+	1    9250 1700
+	-1   0    0    -1
+$EndComp
+$Comp
+L Connector:RJ10 J2
+U 1 1 5C3ED1FE
+P 9250 3000
+F 0 "J2" H 8920 3096 50  0000 R CNN
+F 1 "RJ10" H 8920 3005 50  0000 R CNN
+F 2 "Local_lib:RJ14" V 9250 3050 50  0001 C CNN
+F 3 "~" V 9250 3050 50  0001 C CNN
+	1    9250 3000
+	-1   0    0    -1
+$EndComp
+$Comp
+L Connector:RJ10 J3
+U 1 1 5C3ED6D8
+P 9250 4300
+F 0 "J3" H 8920 4396 50  0000 R CNN
+F 1 "RJ10" H 8920 4305 50  0000 R CNN
+F 2 "Local_lib:RJ14" V 9250 4350 50  0001 C CNN
+F 3 "~" V 9250 4350 50  0001 C CNN
+	1    9250 4300
+	-1   0    0    -1
+$EndComp
+$Comp
+L Connector:RJ10 J4
+U 1 1 5C3ED8E8
+P 9250 5600
+F 0 "J4" H 8920 5696 50  0000 R CNN
+F 1 "RJ10" H 8920 5605 50  0000 R CNN
+F 2 "Local_lib:RJ14" V 9250 5650 50  0001 C CNN
+F 3 "~" V 9250 5650 50  0001 C CNN
+	1    9250 5600
+	-1   0    0    -1
+$EndComp
+$Comp
+L Connector_Generic:Conn_02x20_Odd_Even J5
+U 1 1 5C3F1F55
+P 3300 3700
+F 0 "J5" H 3350 2475 50  0000 C CNN
+F 1 "Conn_02x20_Odd_Even" H 3350 2566 50  0000 C CNN
+F 2 "Connector_PinSocket_2.54mm:PinSocket_2x20_P2.54mm_Vertical" H 3300 3700 50  0001 C CNN
+F 3 "~" H 3300 3700 50  0001 C CNN
+	1    3300 3700
+	-1   0    0    1
+$EndComp
+Connection ~ 3500 2700
 $EndSCHEMATC

Commit message: Partial updates to PiZero integration.
Connections:
- wire segments 93 -> 90
- no-connect marks 23 -> 21
Other:
- moved on the sheet: D1
Changed lines of the file:
@@
 Text Label 6050 5500 0    60   ~ 0
 C_LOAD
-NoConn ~ 3500 4600
-NoConn ~ 3500 4500
-NoConn ~ 3500 4400
-NoConn ~ 3500 4300
-NoConn ~ 3500 4200
-NoConn ~ 3500 4100
 NoConn ~ 3500 4000
-NoConn ~ 3500 3900
-NoConn ~ 3500 3800
-NoConn ~ 3500 3700
-NoConn ~ 3500 3600
-NoConn ~ 3500 3500
-NoConn ~ 3500 3400
-NoConn ~ 3500 3300
-NoConn ~ 3500 3200
-NoConn ~ 3500 3100
-NoConn ~ 3500 3000
 NoConn ~ 3000 3500
 NoConn ~ 3000 2700
-NoConn ~ 3500 2900
 NoConn ~ 3000 4000
 NoConn ~ 3000 4100
@@
 L power:GND #PWR08
 U 1 1 5B4F3E4D
-P 2600 3100
-F 0 "#PWR08" H 2600 2850 50  0001 C CNN
-F 1 "GND" H 2600 2950 50  0000 C CNN
-F 2 "" H 2600 3100 50  0001 C CNN
-F 3 "" H 2600 3100 50  0001 C CNN
-	1    2600 3100
-	0    1    -1   0
+P 3500 2900
+F 0 "#PWR08" H 3500 2650 50  0001 C CNN
+F 1 "GND" H 3500 2750 50  0000 C CNN
+F 2 "" H 3500 2900 50  0001 C CNN
+F 3 "" H 3500 2900 50  0001 C CNN
+	1    3500 2900
+	0    -1   1    0
 $EndComp
 NoConn ~ 3000 4300
@@
 	1    0    0    -1
 $EndComp
-Wire Wire Line
-	2600 3100 3000 3100
 $Comp
 L power:GND #PWR09
@@
 	1    0    0    -1
 $EndComp
-Connection ~ 3800 2700
+Connection ~ 4350 2700
 $Comp
 L PiKwonDo:SN74LV1T34DBVR U2
@@
 L power:+5V #PWR012
 U 1 1 5B5B749D
-P 3800 2650
-F 0 "#PWR012" H 3800 2500 50  0001 C CNN
-F 1 "+5V" H 3800 2790 50  0000 C CNN
-F 2 "" H 3800 2650 50  0001 C CNN
-F 3 "" H 3800 2650 50  0001 C CNN
-	1    3800 2650
+P 4350 2650
+F 0 "#PWR012" H 4350 2500 50  0001 C CNN
+F 1 "+5V" H 4350 2790 50  0000 C CNN
+F 2 "" H 4350 2650 50  0001 C CNN
+F 3 "" H 4350 2650 50  0001 C CNN
+	1    4350 2650
 	-1   0    0    -1
 $EndComp
@@
 L power:GND #PWR014
 U 1 1 5B5B48CC
-P 3800 3050
-F 0 "#PWR014" H 3800 2800 50  0001 C CNN
-F 1 "GND" H 3800 2900 50  0000 C CNN
-F 2 "" H 3800 3050 50  0001 C CNN
-F 3 "" H 3800 3050 50  0001 C CNN
-	1    3800 3050
+P 4350 3050
+F 0 "#PWR014" H 4350 2800 50  0001 C CNN
+F 1 "GND" H 4350 2900 50  0000 C CNN
+F 2 "" H 4350 3050 50  0001 C CNN
+F 3 "" H 4350 3050 50  0001 C CNN
+	1    4350 3050
 	-1   0    0    -1
 $EndComp
 Wire Wire Line
-	3500 2700 3800 2700
-Wire Wire Line
-	3800 2650 3800 2700
+	3500 2700 4350 2700
+Wire Wire Line
+	4350 2650 4350 2700
 Wire Wire Line
 	3500 2800 3500 2700
 Text Label 6050 1700 0    60   ~ 0
 J1_DATA
-Wire Wire Line
-	3000 2800 2600 2800
-Wire Wire Line
-	3000 2900 2600 2900
-Text Label 2600 3000 0    60   ~ 0
+Text Label 3750 4400 0    60   ~ 0
 J1_DATA
-Text Label 2600 2900 0    60   ~ 0
+Text Label 3750 4500 0    60   ~ 0
 J1_LOAD
 Text Label 6050 3000 0    60   ~ 0
@@
 Text Label 6050 5600 0    60   ~ 0
 C_DATA
-Wire Wire Line
-	3000 3200 2600 3200
-Wire Wire Line
-	3000 3300 2600 3300
-Text Label 2600 3400 0    60   ~ 0
+Text Label 3750 3800 0    60   ~ 0
 J2_DATA
-Text Label 2600 3300 0    60   ~ 0
+Text Label 3750 3900 0    60   ~ 0
 J2_LOAD
-Wire Wire Line
-	3000 3000 2600 3000
-Text Label 2600 2800 0    60   ~ 0
+Text Label 3750 4600 0    60   ~ 0
 J1_CLK
-Wire Wire Line
-	3000 3400 2600 3400
-Text Label 2600 3200 0    60   ~ 0
+Text Label 3750 4200 0    60   ~ 0
 J2_CLK
-$Comp
-L power:GND #PWR016
-U 1 1 5B5CF1A3
-P 2600 3900
-F 0 "#PWR016" H 2600 3650 50  0001 C CNN
-F 1 "GND" H 2600 3750 50  0000 C CNN
-F 2 "" H 2600 3900 50  0001 C CNN
-F 3 "" H 2600 3900 50  0001 C CNN
-	1    2600 3900
-	0    1    -1   0
-$EndComp
-Wire Wire Line
-	3000 3600 2600 3600
-Wire Wire Line
-	3000 3700 2600 3700
-Text Label 2600 3800 0    60   ~ 0
+Text Label 3750 3400 0    60   ~ 0
 J3_DATA
-Text Label 2600 3700 0    60   ~ 0
+Text Label 3750 3500 0    60   ~ 0
 J3_LOAD
-Wire Wire Line
-	3000 3800 2600 3800
-Text Label 2600 3600 0    60   ~ 0
+Text Label 4250 3950 0    60   ~ 0
 J3_CLK
-Wire Wire Line
-	2600 3900 3000 3900
-Wire Wire Line
-	3000 4200 2600 4200
-Text Label 2600 4200 0    60   ~ 0
+Text Label 3750 3200 0    60   ~ 0
 C_CLK
-Wire Wire Line
-	3000 4400 2600 4400
-Text Label 2600 4500 0    60   ~ 0
+Text Label 3750 3000 0    60   ~ 0
 C_DATA
-Text Label 2600 4400 0    60   ~ 0
+Text Label 3750 3100 0    60   ~ 0
 C_LOAD
-Wire Wire Line
-	3000 4500 2600 4500
-$Comp
-L power:GND #PWR017
-U 1 1 5B5CF526
-P 2600 4600
-F 0 "#PWR017" H 2600 4350 50  0001 C CNN
-F 1 "GND" H 2600 4450 50  0000 C CNN
-F 2 "" H 2600 4600 50  0001 C CNN
-F 3 "" H 2600 4600 50  0001 C CNN
-	1    2600 4600
-	0    1    -1   0
-$EndComp
-Wire Wire Line
-	2600 4600 3000 4600
 $Comp
 L power:GND #PWR018
@@
 L Device:D_Zener D1
 U 1 1 5B5DD772
-P 3800 2900
-F 0 "D1" V 3700 2925 50  0000 L CNN
-F 1 "5V" V 3900 2925 50  0000 L CNN
-F 2 "Diodes_SMD:D_SOD-323_HandSoldering" H 3800 2900 50  0001 C CNN
-F 3 "" H 3800 2900 50  0001 C CNN
-	1    3800 2900
+P 4350 2900
+F 0 "D1" V 4250 2925 50  0000 L CNN
+F 1 "5V" V 4450 2925 50  0000 L CNN
+F 2 "Diodes_SMD:D_SOD-323_HandSoldering" H 4350 2900 50  0001 C CNN
+F 3 "" H 4350 2900 50  0001 C CNN
+	1    4350 2900
 	0    1    1    0
 $EndComp
@@
 	8000 5500 8850 5500
 Wire Wire Line
-	3800 2700 3800 2750
+	4350 2700 4350 2750
 Wire Wire Line
 	6750 1700 7400 1700
@@
 $EndComp
 Connection ~ 3500 2700
+$Comp
+L power:GND #PWR0101
+U 1 1 5C7A81B9
+P 3500 3300
+F 0 "#PWR0101" H 3500 3050 50  0001 C CNN
+F 1 "GND" H 3500 3150 50  0000 C CNN
+F 2 "" H 3500 3300 50  0001 C CNN
+F 3 "" H 3500 3300 50  0001 C CNN
+	1    3500 3300
+	0    -1   1    0
+$EndComp
+$Comp
+L power:GND #PWR0102
+U 1 1 5C7AAEDE
+P 3500 3600
+F 0 "#PWR0102" H 3500 3350 50  0001 C CNN
+F 1 "GND" H 3500 3450 50  0000 C CNN
+F 2 "" H 3500 3600 50  0001 C CNN
+F 3 "" H 3500 3600 50  0001 C CNN
+	1    3500 3600
+	0    -1   1    0
+$EndComp
+$Comp
+L power:GND #PWR0103
+U 1 1 5C7AB267
+P 3500 4100
+F 0 "#PWR0103" H 3500 3850 50  0001 C CNN
+F 1 "GND" H 3500 3950 50  0000 C CNN
+F 2 "" H 3500 4100 50  0001 C CNN
+F 3 "" H 3500 4100 50  0001 C CNN
+	1    3500 4100
+	0    -1   1    0
+$EndComp
+$Comp
+L power:GND #PWR0104
+U 1 1 5C7AB2C6
+P 3500 4300
+F 0 "#PWR0104" H 3500 4050 50  0001 C CNN
+F 1 "GND" H 3500 4150 50  0000 C CNN
+F 2 "" H 3500 4300 50  0001 C CNN
+F 3 "" H 3500 4300 50  0001 C CNN
+	1    3500 4300
+	0    -1   1    0
+$EndComp
+NoConn ~ 3000 2800
+NoConn ~ 3000 2900
+NoConn ~ 3000 3000
+NoConn ~ 3000 3100
+NoConn ~ 3000 3200
+NoConn ~ 3000 3300
+NoConn ~ 3000 3400
+NoConn ~ 3000 3600
+NoConn ~ 3000 3700
+NoConn ~ 3000 3800
+NoConn ~ 3000 3900
+NoConn ~ 3000 4200
+NoConn ~ 3000 4400
+NoConn ~ 3000 4500
+NoConn ~ 3000 4600
+Wire Wire Line
+	3750 3000 3500 3000
+Wire Wire Line
+	3500 3100 3750 3100
+Wire Wire Line
+	3750 3200 3500 3200
+Wire Wire Line
+	3500 3400 3750 3400
+Wire Wire Line
+	3750 3500 3500 3500
+Wire Wire Line
+	3500 3700 3750 3700
+Wire Wire Line
+	3750 3800 3500 3800
+Wire Wire Line
+	3500 3900 3750 3900
+Wire Wire Line
+	3750 4200 3500 4200
+Wire Wire Line
+	3500 4400 3750 4400
+Wire Wire Line
+	3750 4500 3500 4500
+Wire Wire Line
+	3500 4600 3750 4600
 $EndSCHEMATC
