File: Electronics/PiKwonDoHAT/PiKwonDoHAT.sch (KiCad schematic (older format))
At the start: 42 parts, among them J1 RJ10, J2 RJ10, J3 RJ10, J4 RJ10, J5 Conn_02x20_Odd_Even, U1 74LV1T34, U2 74LV1T34, U3 74LV1T34, U4 74LV1T34

Commit message: Updated to mate with RasPi Zero, reduced footprint significantly.
Parts:
- U1, U2, U3, U4: symbol PiKwonDo:SN74LV1T34DBVR -> PiKwonDoHAT-rescue:SN74LV1T34DBVR-PiKwonDo
Connections:
- no-connect marks 21 -> 20
Changed lines of the file:
@@
 NoConn ~ 3000 4300
 $Comp
-L PiKwonDo:SN74LV1T34DBVR U1
+L PiKwonDoHAT-rescue:SN74LV1T34DBVR-PiKwonDo U1
 U 1 1 5B5B2161
 P 5500 1400
@@
 Connection ~ 4350 2700
 $Comp
-L PiKwonDo:SN74LV1T34DBVR U2
+L PiKwonDoHAT-rescue:SN74LV1T34DBVR-PiKwonDo U2
 U 1 1 5B5B4D01
 P 5650 2850
@@
 Text Label 6050 1700 0    60   ~ 0
 J1_DATA
-Text Label 3750 4400 0    60   ~ 0
+Text Label 3750 4500 0    60   ~ 0
 J1_DATA
-Text Label 3750 4500 0    60   ~ 0
+Text Label 3750 4600 0    60   ~ 0
 J1_LOAD
 Text Label 6050 3000 0    60   ~ 0
@@
 Text Label 6050 5600 0    60   ~ 0
 C_DATA
+Text Label 3750 3900 0    60   ~ 0
+J2_DATA
+Text Label 3750 4200 0    60   ~ 0
+J2_LOAD
+Text Label 3750 4400 0    60   ~ 0
+J1_CLK
 Text Label 3750 3800 0    60   ~ 0
-J2_DATA
-Text Label 3750 3900 0    60   ~ 0
-J2_LOAD
-Text Label 3750 4600 0    60   ~ 0
-J1_CLK
-Text Label 3750 4200 0    60   ~ 0
 J2_CLK
+Text Label 3750 3500 0    60   ~ 0
+J3_DATA
+Text Label 3750 3700 0    60   ~ 0
+J3_LOAD
 Text Label 3750 3400 0    60   ~ 0
-J3_DATA
-Text Label 3750 3500 0    60   ~ 0
-J3_LOAD
-Text Label 4250 3950 0    60   ~ 0
 J3_CLK
+Text Label 3750 3000 0    60   ~ 0
+C_CLK
+Text Label 3750 3100 0    60   ~ 0
+C_DATA
 Text Label 3750 3200 0    60   ~ 0
-C_CLK
-Text Label 3750 3000 0    60   ~ 0
-C_DATA
-Text Label 3750 3100 0    60   ~ 0
 C_LOAD
 $Comp
@@
 	7400 4100 6050 4100
 $Comp
-L PiKwonDo:SN74LV1T34DBVR U3
+L PiKwonDoHAT-rescue:SN74LV1T34DBVR-PiKwonDo U3
 U 1 1 5B5DA6CA
 P 5650 4150
@@
 $EndComp
 $Comp
-L PiKwonDo:SN74LV1T34DBVR U4
+L PiKwonDoHAT-rescue:SN74LV1T34DBVR-PiKwonDo U4
 U 1 1 5B5DA6D6
 P 5650 5450
@@
 NoConn ~ 3000 4400
 NoConn ~ 3000 4500
-NoConn ~ 3000 4600
 Wire Wire Line
 	3750 3000 3500 3000
@@
 Wire Wire Line
 	3500 4600 3750 4600
+$Comp
+L power:GND #PWR?
+U 1 1 5C7A38CB
+P 3000 4600
+F 0 "#PWR?" H 3000 4350 50  0001 C CNN
+F 1 "GND" H 3000 4450 50  0000 C CNN
+F 2 "" H 3000 4600 50  0001 C CNN
+F 3 "" H 3000 4600 50  0001 C CNN
+	1    3000 4600
+	0    1    -1   0
+$EndComp
 $EndSCHEMATC

Commit message: Updated boards for two-sided manufacture.
Parts:
- C1, C10, C11, C12, C2, C3, C4, C5, C6, C7, C8, C9: symbol Device:C -> PiKwonDoHAT-rescue:C-Device
- D1, D2, D3, D4, D5, D6, D7, D8, D9: symbol Device:D_Zener -> PiKwonDoHAT-rescue:D_Zener-Device
- J1, J2, J3, J4: symbol Connector:RJ10 -> PiKwonDoHAT-rescue:RJ10-Connector
- J5: symbol Connector_Generic:Conn_02x20_Odd_Even -> PiKwonDoHAT-rescue:Conn_02x20_Odd_Even-Connector_Generic
- R1, R10, R11, R12, R2, R3, R4, R5, R6, R7, R8, R9: symbol Device:R -> PiKwonDoHAT-rescue:R-Device
