File: Electronics/Timer/Timer.sch (KiCad schematic (older format))
At the start: 21 parts, among them CN1 RJ12-UNSHLD, U1 MIC5504-3.3YM5, U2 74HC165

Commit message: Synchronized PCB with new netlist; cleaned up glitches.
Parts:
- U2: footprint (none) -> Housings_DIP:DIP-16_W7.62mm
Changed lines of the file:
@@
 Sheet 1 1
 Title ""
-Date ""
+Date "2018-7-29 (#1)"
 Rev ""
 Comp ""
@@
 	1    0    0    -1
 $EndComp
-Wire Wire Line
-	1450 1550 1450 1500
 $Comp
 L R_Network05 RN1
@@
 NoConn ~ 9300 5000
 NoConn ~ 9300 5900
-Wire Wire Line
-	9100 1300 9100 2750
-Wire Wire Line
-	9100 2000 8300 2000
-Wire Wire Line
-	9000 1300 9000 3650
-Wire Wire Line
-	9000 2150 8300 2150
-Wire Wire Line
-	8900 1300 8900 4550
-Wire Wire Line
-	8900 2300 8300 2300
-Wire Wire Line
-	8800 1300 8800 5450
-Wire Wire Line
-	9200 1300 9200 1850
-Wire Wire Line
-	8300 2900 8800 2900
-Connection ~ 8800 2900
 $Comp
 L R R1
@@
 F 0 "U2" H 7700 2550 60  0000 C CNN
 F 1 "74HC165" H 7700 2200 60  0000 C CNN
-F 2 "" H 7700 2200 60  0001 C CNN
+F 2 "Housings_DIP:DIP-16_W7.62mm" H 7700 2200 60  0001 C CNN
 F 3 "" H 7700 2200 60  0001 C CNN
 	1    7700 2200
 	-1   0    0    -1
 $EndComp
-Wire Wire Line
-	2000 3300 3050 3300
-Wire Wire Line
-	7700 950  7700 1050
-Connection ~ 7700 1000
-Wire Wire Line
-	7700 1000 7850 1000
-Wire Wire Line
-	3350 3300 3650 3300
-Wire Wire Line
-	4250 3850 4250 3750
-Wire Wire Line
-	4250 3450 4250 3300
-Wire Wire Line
-	3950 3300 5000 3300
-Wire Wire Line
-	4600 3300 4600 3450
-Connection ~ 4250 3300
-Connection ~ 4600 3300
 $Comp
 L GND #PWR?
@@
 	-1   0    0    -1
 $EndComp
-Wire Wire Line
-	4600 3850 4600 3750
 $Comp
 L GND #PWR?
@@
 	-1   0    0    -1
 $EndComp
-Wire Wire Line
-	5350 4250 5350 4100
 $Comp
 L +5V #PWR?
@@
 	0    1    1    0
 $EndComp
-Wire Wire Line
-	4950 3700 4900 3700
-Wire Wire Line
-	4900 3700 4900 3300
-Connection ~ 4900 3300
 $Comp
 L +5V #PWR?
@@
 	0    1    1    0
 $EndComp
-Wire Wire Line
-	5750 3900 5800 3900
-Wire Wire Line
-	5750 3700 6300 3700
-Wire Wire Line
-	6200 3850 6200 3700
-Connection ~ 6200 3700
-Wire Wire Line
-	6200 4250 6200 4150
 $Comp
 L D_Zener D4
@@
 $Comp
 L GND #PWR?
-U 1 1 5B5E675F
-P 8300 2450
-F 0 "#PWR?" H 8300 2200 50  0001 C CNN
-F 1 "GND" H 8300 2300 50  0000 C CNN
-F 2 "" H 8300 2450 50  0001 C CNN
-F 3 "" H 8300 2450 50  0001 C CNN
-	1    8300 2450
-	0    -1   1    0
-$EndComp
-$Comp
-L GND #PWR?
 U 1 1 5B5E67AC
 P 8300 2600
@@
 	0    1    -1   0
 $EndComp
-Wire Wire Line
-	3050 3700 2900 3700
-Wire Wire Line
-	2900 3300 2900 4100
-Connection ~ 2900 3300
 $Comp
 L GND #PWR?
@@
 	0    -1   1    0
 $EndComp
-Wire Wire Line
-	3850 3700 3750 3700
-Wire Wire Line
-	3450 3700 3350 3700
 $Comp
 L R R3
@@
 	0    1    -1   0
 $EndComp
-Wire Wire Line
-	2900 4100 3050 4100
-Connection ~ 2900 3700
 Text Label 3700 4500 2    60   ~ 0
 ~LOAD~
-Wire Wire Line
-	3350 4100 3700 4100
-Wire Wire Line
-	3050 4500 2800 4500
-Wire Wire Line
-	2800 4500 2800 3400
-Wire Wire Line
-	2800 3400 2000 3400
 Text Label 3700 4100 2    60   ~ 0
 CLK
-Wire Wire Line
-	3350 4500 3700 4500
 $Comp
 L C C3
@@
 	-1   0    0    -1
 $EndComp
-Wire Wire Line
-	2200 4100 2400 4100
-Wire Wire Line
-	2400 3500 2400 4250
 $Comp
 L GND #PWR?
@@
 	-1   0    0    -1
 $EndComp
-Wire Wire Line
-	2400 4650 2400 4550
 Text Label 1650 4100 0    60   ~ 0
 Q
-Wire Wire Line
-	1650 4100 1900 4100
-Wire Wire Line
-	2400 3500 2000 3500
-Connection ~ 2400 4100
 $Comp
 L R R4
@@
 	0    1    -1   0
 $EndComp
-Wire Wire Line
-	8300 1400 8550 1400
 Text Label 8550 1400 2    60   ~ 0
 Q
 Text Label 6750 1550 0    60   ~ 0
 ~LOAD~
-Wire Wire Line
-	7100 1400 6750 1400
 Text Label 6750 1400 0    60   ~ 0
 CLK
-Wire Wire Line
-	7100 1550 6750 1550
 $Comp
 L GND #PWR?
@@
 	0    1    -1   0
 $EndComp
-Wire Wire Line
-	8300 1850 9300 1850
-Connection ~ 9100 2000
-Connection ~ 9000 2150
-Connection ~ 8900 2300
 $Comp
 L GND #PWR?
@@
 	0    -1   1    0
 $EndComp
+$Comp
+L +3.3V #PWR?
+U 1 1 5B5E2650
+P 8300 2450
+F 0 "#PWR?" H 8300 2300 50  0001 C CNN
+F 1 "+3.3V" V 8300 2700 50  0000 C CNN
+F 2 "" H 8300 2450 50  0001 C CNN
+F 3 "" H 8300 2450 50  0001 C CNN
+	1    8300 2450
+	0    1    -1   0
+$EndComp
+Wire Wire Line
+	1450 1550 1450 1500
+Wire Wire Line
+	9100 1300 9100 2750
+Wire Wire Line
+	9100 2000 8300 2000
+Wire Wire Line
+	9000 1300 9000 3650
+Wire Wire Line
+	9000 2150 8300 2150
+Wire Wire Line
+	8900 1300 8900 4550
+Wire Wire Line
+	8900 2300 8300 2300
+Wire Wire Line
+	8800 1300 8800 5450
+Wire Wire Line
+	9200 1300 9200 1850
+Wire Wire Line
+	8300 2900 8800 2900
+Connection ~ 8800 2900
+Wire Wire Line
+	2000 3300 3050 3300
+Wire Wire Line
+	7700 950  7700 1050
+Connection ~ 7700 1000
+Wire Wire Line
+	7700 1000 7850 1000
+Wire Wire Line
+	3350 3300 3650 3300
+Wire Wire Line
+	4250 3850 4250 3750
+Wire Wire Line
+	4250 3450 4250 3300
+Wire Wire Line
+	3950 3300 5000 3300
+Wire Wire Line
+	4600 3300 4600 3450
+Connection ~ 4250 3300
+Connection ~ 4600 3300
+Wire Wire Line
+	4600 3850 4600 3750
+Wire Wire Line
+	5350 4250 5350 4100
+Wire Wire Line
+	4950 3700 4900 3700
+Wire Wire Line
+	4900 3700 4900 3300
+Connection ~ 4900 3300
+Wire Wire Line
+	5750 3900 5800 3900
+Wire Wire Line
+	5750 3700 6300 3700
+Wire Wire Line
+	6200 3850 6200 3700
+Connection ~ 6200 3700
+Wire Wire Line
+	6200 4250 6200 4150
+Wire Wire Line
+	3050 3700 2900 3700
+Wire Wire Line
+	2900 3300 2900 4100
+Connection ~ 2900 3300
+Wire Wire Line
+	3850 3700 3750 3700
+Wire Wire Line
+	3450 3700 3350 3700
+Wire Wire Line
+	2900 4100 3050 4100
+Connection ~ 2900 3700
+Wire Wire Line
+	3350 4100 3700 4100
+Wire Wire Line
+	3050 4500 2800 4500
+Wire Wire Line
+	2800 4500 2800 3400
+Wire Wire Line
+	2800 3400 2000 3400
+Wire Wire Line
+	3350 4500 3700 4500
+Wire Wire Line
+	2200 4100 2400 4100
+Wire Wire Line
+	2400 3500 2400 4250
+Wire Wire Line
+	2400 4650 2400 4550
+Wire Wire Line
+	1650 4100 1900 4100
+Wire Wire Line
+	2400 3500 2000 3500
+Connection ~ 2400 4100
+Wire Wire Line
+	8300 1400 8550 1400
+Wire Wire Line
+	7100 1400 6750 1400
+Wire Wire Line
+	7100 1550 6750 1550
+Wire Wire Line
+	8300 1850 9300 1850
+Connection ~ 9100 2000
+Connection ~ 9000 2150
+Connection ~ 8900 2300
 Connection ~ 9200 1850
 Wire Wire Line

Commit message: Timer: Rerouted to eliminate jumpers, at the cost of a few 1206's with two traces underneath.
Parts:
- added R6: 470, Resistors_SMD:R_1206_HandSoldering, symbol R
Connections:
- wire segments 49 -> 51
- no-connect marks 23 -> 24
Changed lines of the file:
@@
 L R_Network05 RN1
 U 1 1 5B2D83AE
-P 9000 1100
-F 0 "RN1" V 8700 1100 50  0000 C CNN
-F 1 "5x 47k" H 9000 1300 50  0000 C CNN
-F 2 "Resistors_THT:R_Array_SIP6" V 9375 1100 50  0001 C CNN
-F 3 "" H 9000 1100 50  0001 C CNN
-	1    9000 1100
-	-1   0    0    -1
+P 9100 1100
+F 0 "RN1" V 8800 1100 50  0000 C CNN
+F 1 "5x 47k" H 9100 1300 50  0000 C CNN
+F 2 "Resistors_THT:R_Array_SIP6" V 9475 1100 50  0001 C CNN
+F 3 "" H 9100 1100 50  0001 C CNN
+	1    9100 1100
+	1    0    0    -1
 $EndComp
 $Comp
@@
 $EndComp
 $Comp
-L GND #PWR05
+L GND #PWR04
 U 1 1 5B2D939C
 P 2000 3600
-F 0 "#PWR05" H 2000 3350 50  0001 C CNN
+F 0 "#PWR04" H 2000 3350 50  0001 C CNN
 F 1 "GND" H 2000 3450 50  0000 C CNN
 F 2 "" H 2000 3600 50  0001 C CNN
@@
 NoConn ~ 8300 1550
 $Comp
-L GND #PWR06
+L GND #PWR05
 U 1 1 5B2D93FE
 P 7700 3250
-F 0 "#PWR06" H 7700 3000 50  0001 C CNN
+F 0 "#PWR05" H 7700 3000 50  0001 C CNN
 F 1 "GND" H 7700 3100 50  0000 C CNN
 F 2 "" H 7700 3250 50  0001 C CNN
@@
 $EndComp
 $Comp
-L GND #PWR07
+L GND #PWR06
 U 1 1 5B2D95FE
 P 8150 1000
-F 0 "#PWR07" H 8150 750 50  0001 C CNN
+F 0 "#PWR06" H 8150 750 50  0001 C CNN
 F 1 "GND" H 8150 850 50  0000 C CNN
 F 2 "" H 8150 1000 50  0001 C CNN
@@
 $EndComp
 $Comp
-L +3.3V #PWR08
+L +3.3V #PWR07
 U 1 1 5B2D9621
 P 7700 950
-F 0 "#PWR08" H 7700 800 50  0001 C CNN
+F 0 "#PWR07" H 7700 800 50  0001 C CNN
 F 1 "+3.3V" H 7700 1090 50  0000 C CNN
 F 2 "" H 7700 950 50  0001 C CNN
 F 3 "" H 7700 950 50  0001 C CNN
 	1    7700 950
-	-1   0    0    -1
-$EndComp
-$Comp
-L +3.3V #PWR09
-U 1 1 5B2D9644
-P 9200 900
-F 0 "#PWR09" H 9200 750 50  0001 C CNN
-F 1 "+3.3V" H 9200 1040 50  0000 C CNN
-F 2 "" H 9200 900 50  0001 C CNN
-F 3 "" H 9200 900 50  0001 C CNN
-	1    9200 900
 	-1   0    0    -1
 $EndComp
@@
 NoConn ~ 10400 6000
 $Comp
-L GND #PWR011
+L GND #PWR08
 U 1 1 5B2DA1C3
 P 10400 1950
-F 0 "#PWR011" H 10400 1700 50  0001 C CNN
+F 0 "#PWR08" H 10400 1700 50  0001 C CNN
 F 1 "GND" H 10400 1800 50  0000 C CNN
 F 2 "" H 10400 1950 50  0001 C CNN
@@
 $EndComp
 $Comp
-L GND #PWR012
+L GND #PWR09
 U 1 1 5B2DA234
 P 10400 2850
-F 0 "#PWR012" H 10400 2600 50  0001 C CNN
+F 0 "#PWR09" H 10400 2600 50  0001 C CNN
 F 1 "GND" H 10400 2700 50  0000 C CNN
 F 2 "" H 10400 2850 50  0001 C CNN
@@
 $EndComp
 $Comp
-L GND #PWR016
+L GND #PWR010
 U 1 1 5B46CF5B
 P 4250 3850
-F 0 "#PWR016" H 4250 3600 50  0001 C CNN
+F 0 "#PWR010" H 4250 3600 50  0001 C CNN
 F 1 "GND" H 4250 3700 50  0000 C CNN
 F 2 "" H 4250 3850 50  0001 C CNN
@@
 $EndComp
 $Comp
-L GND #PWR019
+L GND #PWR011
 U 1 1 5B5B72D4
 P 6200 4250
-F 0 "#PWR019" H 6200 4000 50  0001 C CNN
+F 0 "#PWR011" H 6200 4000 50  0001 C CNN
 F 1 "GND" H 6200 4100 50  0000 C CNN
 F 2 "" H 6200 4250 50  0001 C CNN
@@
 $EndComp
 $Comp
-L GND #PWR?
+L GND #PWR012
 U 1 1 5B5E52E5
 P 4600 3850
-F 0 "#PWR?" H 4600 3600 50  0001 C CNN
+F 0 "#PWR012" H 4600 3600 50  0001 C CNN
 F 1 "GND" H 4600 3700 50  0000 C CNN
 F 2 "" H 4600 3850 50  0001 C CNN
@@
 $EndComp
 $Comp
-L GND #PWR?
+L GND #PWR013
 U 1 1 5B5E531A
 P 5350 4250
-F 0 "#PWR?" H 5350 4000 50  0001 C CNN
+F 0 "#PWR013" H 5350 4000 50  0001 C CNN
 F 1 "GND" H 5350 4100 50  0000 C CNN
 F 2 "" H 5350 4250 50  0001 C CNN
@@
 $EndComp
 $Comp
-L +5V #PWR?
+L +5V #PWR014
 U 1 1 5B5E5952
 P 5000 3300
-F 0 "#PWR?" H 5000 3150 50  0001 C CNN
+F 0 "#PWR014" H 5000 3150 50  0001 C CNN
 F 1 "+5V" H 5000 3440 50  0000 C CNN
 F 2 "" H 5000 3300 50  0001 C CNN
@@
 $EndComp
 $Comp
-L +5V #PWR?
+L +5V #PWR015
 U 1 1 5B5E5C2E
 P 5800 3900
-F 0 "#PWR?" H 5800 3750 50  0001 C CNN
+F 0 "#PWR015" H 5800 3750 50  0001 C CNN
 F 1 "+5V" H 5800 4040 50  0000 C CNN
 F 2 "" H 5800 3900 50  0001 C CNN
@@
 $EndComp
 $Comp
-L GND #PWR?
+L GND #PWR016
 U 1 1 5B5E67AC
 P 8300 2600
-F 0 "#PWR?" H 8300 2350 50  0001 C CNN
+F 0 "#PWR016" H 8300 2350 50  0001 C CNN
 F 1 "GND" H 8300 2450 50  0000 C CNN
 F 2 "" H 8300 2600 50  0001 C CNN
@@
 $EndComp
 $Comp
-L GND #PWR?
+L GND #PWR017
 U 1 1 5B5E67F9
 P 8300 2750
-F 0 "#PWR?" H 8300 2500 50  0001 C CNN
+F 0 "#PWR017" H 8300 2500 50  0001 C CNN
 F 1 "GND" H 8300 2600 50  0000 C CNN
 F 2 "" H 8300 2750 50  0001 C CNN
@@
 $EndComp
 $Comp
-L GND #PWR?
+L GND #PWR018
 U 1 1 5B5E6846
 P 7100 1850
-F 0 "#PWR?" H 7100 1600 50  0001 C CNN
+F 0 "#PWR018" H 7100 1600 50  0001 C CNN
 F 1 "GND" H 7100 1700 50  0000 C CNN
 F 2 "" H 7100 1850 50  0001 C CNN
@@
 $EndComp
 $Comp
-L GND #PWR?
+L GND #PWR019
 U 1 1 5B5E781E
 P 3850 3700
-F 0 "#PWR?" H 3850 3450 50  0001 C CNN
+F 0 "#PWR019" H 3850 3450 50  0001 C CNN
 F 1 "GND" H 3850 3550 50  0000 C CNN
 F 2 "" H 3850 3700 50  0001 C CNN
@@
 $EndComp
 $Comp
-L GND #PWR?
+L GND #PWR020
 U 1 1 5B5E8FC7
 P 2400 4650
-F 0 "#PWR?" H 2400 4400 50  0001 C CNN
+F 0 "#PWR020" H 2400 4400 50  0001 C CNN
 F 1 "GND" H 2400 4500 50  0000 C CNN
 F 2 "" H 2400 4650 50  0001 C CNN
@@
 CLK
 $Comp
-L GND #PWR?
+L GND #PWR021
 U 1 1 5B5EA020
 P 7100 2900
-F 0 "#PWR?" H 7100 2650 50  0001 C CNN
+F 0 "#PWR021" H 7100 2650 50  0001 C CNN
 F 1 "GND" H 7100 2750 50  0000 C CNN
 F 2 "" H 7100 2900 50  0001 C CNN
@@
 $EndComp
 $Comp
-L GND #PWR?
+L GND #PWR022
 U 1 1 5B5EA568
 P 10400 3750
-F 0 "#PWR?" H 10400 3500 50  0001 C CNN
+F 0 "#PWR022" H 10400 3500 50  0001 C CNN
 F 1 "GND" H 10400 3600 50  0000 C CNN
 F 2 "" H 10400 3750 50  0001 C CNN
@@
 $EndComp
 $Comp
-L GND #PWR?
+L GND #PWR023
 U 1 1 5B5EA5B2
-P 10400 4650
-F 0 "#PWR?" H 10400 4400 50  0001 C CNN
-F 1 "GND" H 10400 4500 50  0000 C CNN
-F 2 "" H 10400 4650 50  0001 C CNN
-F 3 "" H 10400 4650 50  0001 C CNN
-	1    10400 4650
-	0    -1   1    0
-$EndComp
-$Comp
-L GND #PWR?
+P 9300 4550
+F 0 "#PWR023" H 9300 4300 50  0001 C CNN
+F 1 "GND" H 9300 4400 50  0000 C CNN
+F 2 "" H 9300 4550 50  0001 C CNN
+F 3 "" H 9300 4550 50  0001 C CNN
+	1    9300 4550
+	0    1    -1   0
+$EndComp
+$Comp
+L GND #PWR024
 U 1 1 5B5EA5FC
 P 10400 5550
-F 0 "#PWR?" H 10400 5300 50  0001 C CNN
+F 0 "#PWR024" H 10400 5300 50  0001 C CNN
 F 1 "GND" H 10400 5400 50  0000 C CNN
 F 2 "" H 10400 5550 50  0001 C CNN
@@
 $EndComp
 $Comp
-L +3.3V #PWR?
+L +3.3V #PWR025
 U 1 1 5B5E2650
 P 8300 2450
-F 0 "#PWR?" H 8300 2300 50  0001 C CNN
+F 0 "#PWR025" H 8300 2300 50  0001 C CNN
 F 1 "+3.3V" V 8300 2700 50  0000 C CNN
 F 2 "" H 8300 2450 50  0001 C CNN
@@
 	9000 2150 8300 2150
 Wire Wire Line
-	8900 1300 8900 4550
+	8900 1300 8900 4350
 Wire Wire Line
 	8900 2300 8300 2300
 Wire Wire Line
-	8800 1300 8800 5450
+	8800 2900 8800 5450
 Wire Wire Line
 	9200 1300 9200 1850
@@
 	9000 3650 9300 3650
 Wire Wire Line
-	8900 4550 9300 4550
-Wire Wire Line
 	8800 5450 9300 5450
+NoConn ~ 9300 1300
+$Comp
+L R R6
+U 1 1 5B5E2B7E
+P 8800 2750
+F 0 "R6" V 8900 2750 50  0000 C CNN
+F 1 "470" V 8800 2750 50  0000 C CNN
+F 2 "Resistors_SMD:R_1206_HandSoldering" V 8730 2750 50  0001 C CNN
+F 3 "" H 8800 2750 50  0001 C CNN
+	1    8800 2750
+	-1   0    0    -1
+$EndComp
+$Comp
+L +3.3V #PWR026
+U 1 1 5B5E2F61
+P 8800 2600
+F 0 "#PWR026" H 8800 2450 50  0001 C CNN
+F 1 "+3.3V" H 8800 2750 50  0000 C CNN
+F 2 "" H 8800 2600 50  0001 C CNN
+F 3 "" H 8800 2600 50  0001 C CNN
+	1    8800 2600
+	-1   0    0    -1
+$EndComp
+$Comp
+L +5V #PWR027
+U 1 1 5B5E277A
+P 8900 900
+F 0 "#PWR027" H 8900 750 50  0001 C CNN
+F 1 "+5V" H 8900 1040 50  0000 C CNN
+F 2 "" H 8900 900 50  0001 C CNN
+F 3 "" H 8900 900 50  0001 C CNN
+	1    8900 900
+	1    0    0    -1
+$EndComp
+Wire Wire Line
+	10400 4650 10550 4650
+Wire Wire Line
+	10550 4650 10550 4350
+Wire Wire Line
+	10550 4350 8900 4350
 $EndSCHEMATC

Commit message: Timer: Increased C2 to 1 uF (per datasheet for U1 stability); brought RN1 back to 3.3 V instead of 5 V.
Parts:
- C2: value 10nF -> 1uF; footprint Capacitors_SMD:C_0805_HandSoldering -> Capacitors_SMD:C_1206_HandSoldering
Changed lines of the file:
@@
 P 8000 1000
 F 0 "C2" V 8150 1000 50  0000 C CNN
-F 1 "10nF" V 7850 1000 50  0000 C CNN
-F 2 "Capacitors_SMD:C_0805_HandSoldering" H 8038 850 50  0001 C CNN
+F 1 "1uF" V 7850 1000 50  0000 C CNN
+F 2 "Capacitors_SMD:C_1206_HandSoldering" H 8038 850 50  0001 C CNN
 F 3 "" H 8000 1000 50  0001 C CNN
 	1    8000 1000
@@
 	-1   0    0    -1
 $EndComp
-$Comp
-L +5V #PWR027
-U 1 1 5B5E277A
+Wire Wire Line
+	10400 4650 10550 4650
+Wire Wire Line
+	10550 4650 10550 4350
+Wire Wire Line
+	10550 4350 8900 4350
+$Comp
+L +3.3V #PWR?
+U 1 1 5B5E304C
 P 8900 900
-F 0 "#PWR027" H 8900 750 50  0001 C CNN
-F 1 "+5V" H 8900 1040 50  0000 C CNN
+F 0 "#PWR?" H 8900 750 50  0001 C CNN
+F 1 "+3.3V" H 8900 1040 50  0000 C CNN
 F 2 "" H 8900 900 50  0001 C CNN
 F 3 "" H 8900 900 50  0001 C CNN
 	1    8900 900
-	1    0    0    -1
-$EndComp
-Wire Wire Line
-	10400 4650 10550 4650
-Wire Wire Line
-	10550 4650 10550 4350
-Wire Wire Line
-	10550 4350 8900 4350
+	-1   0    0    -1
+$EndComp
 $EndSCHEMATC

Commit message: Updated Timer project to kicad 5
Parts:
- C1, C2, C3: symbol C -> Device:C
- CN1: symbol RJ12-UNSHLD -> PiKwonDo:RJ12-UNSHLD
- D1: symbol D_Schottky -> Device:D_Schottky
- D2: symbol LED -> Device:LED
- D3, D4: symbol D_Zener -> Device:D_Zener
- R1, R2, R3, R4, R5, R6: symbol R -> Device:R
- RN1: symbol R_Network05 -> Device:R_Network05
- S1, S2, S3, S4, S5: symbol DPDT-Button -> Logic_74xx:DPDT-Button
- U1: symbol MIC5504-3.3YM5 -> Timer-rescue:MIC5504-3.3YM5
- U2: symbol 74HC165_PKD -> PiKwonDo:74HC165_PKD
Connections:
- wire segments 51 -> 63
Changed lines of the file:
@@
-EESchema Schematic File Version 2
-LIBS:power
-LIBS:device
-LIBS:switches
-LIBS:relays
-LIBS:motors
-LIBS:transistors
-LIBS:conn
-LIBS:linear
-LIBS:regul
-LIBS:74xx
-LIBS:cmos4000
-LIBS:adc-dac
-LIBS:memory
-LIBS:xilinx
-LIBS:microcontrollers
-LIBS:dsp
-LIBS:microchip
-LIBS:analog_switches
-LIBS:motorola
-LIBS:texas
-LIBS:intel
-LIBS:audio
-LIBS:interface
-LIBS:digital-audio
-LIBS:philips
-LIBS:display
-LIBS:cypress
-LIBS:siliconi
-LIBS:opto
-LIBS:atmel
-LIBS:contrib
-LIBS:valves
-LIBS:Logic_74xx
-LIBS:Logic_CMOS_4000
-LIBS:Logic_CMOS_IEEE
-LIBS:Switch
-LIBS:PiKwonDo
+EESchema Schematic File Version 4
 LIBS:Timer-cache
-EELAYER 25 0
+EELAYER 26 0
 EELAYER END
 $Descr A4 11693 8268
@@
 $EndDescr
 $Comp
-L GND #PWR01
+L power:GND #PWR01
 U 1 1 5B2D833C
 P 1450 1550
@@
 $EndComp
 $Comp
-L PWR_FLAG #FLG02
+L power:PWR_FLAG #FLG02
 U 1 1 5B2D8350
 P 1450 1500
@@
 $EndComp
 $Comp
-L R_Network05 RN1
+L Device:R_Network05 RN1
 U 1 1 5B2D83AE
 P 9100 1100
@@
 $EndComp
 $Comp
-L RJ12-UNSHLD CN1
+L PiKwonDo:RJ12-UNSHLD CN1
 U 1 1 5B2D8F12
 P 1550 3400
@@
 NoConn ~ 2000 3200
 $Comp
-L LED D2
+L Device:LED D2
 U 1 1 5B2D9078
 P 3600 3700
@@
 $EndComp
 $Comp
-L +3.3V #PWR03
+L power:+3.3V #PWR03
 U 1 1 5B2D91A7
 P 6300 3700
@@
 $EndComp
 $Comp
-L GND #PWR04
+L power:GND #PWR04
 U 1 1 5B2D939C
 P 2000 3600
@@
 NoConn ~ 8300 1550
 $Comp
-L GND #PWR05
+L power:GND #PWR05
 U 1 1 5B2D93FE
 P 7700 3250
@@
 $EndComp
 $Comp
-L C C2
+L Device:C C2
 U 1 1 5B2D958C
 P 8000 1000
@@
 $EndComp
 $Comp
-L GND #PWR06
+L power:GND #PWR06
 U 1 1 5B2D95FE
 P 8150 1000
@@
 $EndComp
 $Comp
-L +3.3V #PWR07
+L power:+3.3V #PWR07
 U 1 1 5B2D9621
 P 7700 950
@@
 $EndComp
 $Comp
-L DPDT-Button S5
+L Logic_74xx:DPDT-Button S5
 U 1 1 5B2D9B30
 P 9850 5700
@@
 $EndComp
 $Comp
-L DPDT-Button S1
+L Logic_74xx:DPDT-Button S1
 U 1 1 5B2D9E5E
 P 9850 2100
@@
 $EndComp
 $Comp
-L DPDT-Button S2
+L Logic_74xx:DPDT-Button S2
 U 1 1 5B2D9EA4
 P 9850 3000
@@
 $EndComp
 $Comp
-L DPDT-Button S3
+L Logic_74xx:DPDT-Button S3
 U 1 1 5B2D9EFB
 P 9850 3900
@@
 $EndComp
 $Comp
-L DPDT-Button S4
+L Logic_74xx:DPDT-Button S4
 U 1 1 5B2D9F4B
 P 9850 4800
@@
 NoConn ~ 10400 6000
 $Comp
-L GND #PWR08
+L power:GND #PWR08
 U 1 1 5B2DA1C3
 P 10400 1950
@@
 $EndComp
 $Comp
-L GND #PWR09
+L power:GND #PWR09
 U 1 1 5B2DA234
 P 10400 2850
@@
 NoConn ~ 9300 5900
 $Comp
-L R R1
+L Device:R R1
 U 1 1 5B46CBDD
 P 3200 3300
@@
 $EndComp
 $Comp
-L D_Zener D3
+L Device:D_Zener D3
 U 1 1 5B46CC66
 P 4250 3600
@@
 $EndComp
 $Comp
-L GND #PWR010
+L power:GND #PWR010
 U 1 1 5B46CF5B
 P 4250 3850
@@
 $EndComp
 $Comp
-L MIC5504-3.3YM5 U1
+L Timer-rescue:MIC5504-3.3YM5 U1
 U 1 1 5B5B5636
 P 5350 3800
@@
 $EndComp
 $Comp
-L D_Schottky D1
+L Device:D_Schottky D1
 U 1 1 5B5B5DBA
 P 3800 3300
@@
 $EndComp
 $Comp
-L C C1
+L Device:C C1
 U 1 1 5B5B6007
 P 4600 3600
@@
 $EndComp
 $Comp
-L R R2
+L Device:R R2
 U 1 1 5B5B6D85
 P 3200 3700
@@
 $EndComp
 $Comp
-L GND #PWR011
+L power:GND #PWR011
 U 1 1 5B5B72D4
 P 6200 4250
@@
 $EndComp
 $Comp
-L 74HC165_PKD U2
+L PiKwonDo:74HC165_PKD U2
 U 1 1 5B5E202F
 P 7700 2200
@@
 $EndComp
 $Comp
-L GND #PWR012
+L power:GND #PWR012
 U 1 1 5B5E52E5
 P 4600 3850
@@
 $EndComp
 $Comp
-L GND #PWR013
+L power:GND #PWR013
 U 1 1 5B5E531A
 P 5350 4250
@@
 $EndComp
 $Comp
-L +5V #PWR014
+L power:+5V #PWR014
 U 1 1 5B5E5952
 P 5000 3300
@@
 $EndComp
 $Comp
-L +5V #PWR015
+L power:+5V #PWR015
 U 1 1 5B5E5C2E
 P 5800 3900
@@
 $EndComp
 $Comp
-L D_Zener D4
+L Device:D_Zener D4
 U 1 1 5B5E643D
 P 6200 4000
@@
 $EndComp
 $Comp
-L GND #PWR016
+L power:GND #PWR016
 U 1 1 5B5E67AC
 P 8300 2600
@@
 $EndComp
 $Comp
-L GND #PWR017
+L power:GND #PWR017
 U 1 1 5B5E67F9
 P 8300 2750
@@
 $EndComp
 $Comp
-L GND #PWR018
+L power:GND #PWR018
 U 1 1 5B5E6846
 P 7100 1850
@@
 $EndComp
 $Comp
-L GND #PWR019
+L power:GND #PWR019
 U 1 1 5B5E781E
 P 3850 3700
@@
 $EndComp
 $Comp
-L R R3
+L Device:R R3
 U 1 1 5B5E7B1D
 P 3200 4100
@@
 CLK
 $Comp
-L C C3
+L Device:C C3
 U 1 1 5B5E8ED0
 P 2400 4400
@@
 $EndComp
 $Comp
-L GND #PWR020
+L power:GND #PWR020
 U 1 1 5B5E8FC7
 P 2400 4650
@@
 Q
 $Comp
-L R R4
+L Device:R R4
 U 1 1 5B5E9AEB
 P 3200 4500
@@
 $EndComp
 $Comp
-L R R5
+L Device:R R5
 U 1 1 5B5E9B57
 P 2050 4100
@@
 CLK
 $Comp
-L GND #PWR021
+L power:GND #PWR021
 U 1 1 5B5EA020
 P 7100 2900
@@
 $EndComp
 $Comp
-L GND #PWR022
+L power:GND #PWR022
 U 1 1 5B5EA568
 P 10400 3750
@@
 $EndComp
 $Comp
-L GND #PWR023
+L power:GND #PWR023
 U 1 1 5B5EA5B2
 P 9300 4550
@@
 $EndComp
 $Comp
-L GND #PWR024
+L power:GND #PWR024
 U 1 1 5B5EA5FC
 P 10400 5550
@@
 $EndComp
 $Comp
-L +3.3V #PWR025
+L power:+3.3V #PWR025
 U 1 1 5B5E2650
 P 8300 2450
@@
 	1450 1550 1450 1500
 Wire Wire Line
-	9100 1300 9100 2750
+	9100 1300 9100 2000
 Wire Wire Line
 	9100 2000 8300 2000
 Wire Wire Line
-	9000 1300 9000 3650
+	9000 1300 9000 2150
 Wire Wire Line
 	9000 2150 8300 2150
 Wire Wire Line
-	8900 1300 8900 4350
+	8900 1300 8900 2300
 Wire Wire Line
 	8900 2300 8300 2300
@@
 Connection ~ 8800 2900
 Wire Wire Line
-	2000 3300 3050 3300
-Wire Wire Line
-	7700 950  7700 1050
+	2000 3300 2900 3300
+Wire Wire Line
+	7700 950  7700 1000
 Connection ~ 7700 1000
 Wire Wire Line
@@
 	4250 3450 4250 3300
 Wire Wire Line
-	3950 3300 5000 3300
+	3950 3300 4250 3300
 Wire Wire Line
 	4600 3300 4600 3450
@@
 	5750 3900 5800 3900
 Wire Wire Line
-	5750 3700 6300 3700
+	5750 3700 6200 3700
 Wire Wire Line
 	6200 3850 6200 3700
@@
 	3050 3700 2900 3700
 Wire Wire Line
-	2900 3300 2900 4100
+	2900 3300 2900 3700
 Connection ~ 2900 3300
 Wire Wire Line
@@
 	2200 4100 2400 4100
 Wire Wire Line
-	2400 3500 2400 4250
+	2400 3500 2400 4100
 Wire Wire Line
 	2400 4650 2400 4550
@@
 	7100 1550 6750 1550
 Wire Wire Line
-	8300 1850 9300 1850
+	8300 1850 9200 1850
 Connection ~ 9100 2000
 Connection ~ 9000 2150
@@
 NoConn ~ 9300 1300
 $Comp
-L R R6
+L Device:R R6
 U 1 1 5B5E2B7E
 P 8800 2750
@@
 $EndComp
 $Comp
-L +3.3V #PWR026
+L power:+3.3V #PWR026
 U 1 1 5B5E2F61
 P 8800 2600
@@
 	10550 4350 8900 4350
 $Comp
-L +3.3V #PWR?
+L power:+3.3V #PWR?
 U 1 1 5B5E304C
 P 8900 900
@@
 	-1   0    0    -1
 $EndComp
+Wire Wire Line
+	7700 1000 7700 1050
+Wire Wire Line
+	4250 3300 4600 3300
+Wire Wire Line
+	4600 3300 4900 3300
+Wire Wire Line
+	4900 3300 5000 3300
+Wire Wire Line
+	6200 3700 6300 3700
+Wire Wire Line
+	2900 3300 3050 3300
+Wire Wire Line
+	2900 3700 2900 4100
+Wire Wire Line
+	2400 4100 2400 4250
+Wire Wire Line
+	9100 2000 9100 2750
+Wire Wire Line
+	9000 2150 9000 3650
+Wire Wire Line
+	8900 2300 8900 4350
+Wire Wire Line
+	9200 1850 9300 1850
 $EndSCHEMATC
