File: Electronics/Timer/Timer.sch (KiCad schematic (older format))
At the start: 24 parts, among them J1 RJ10, U1 MIC5504-3.3YM5, U2 74HC165

Commit message: Updated trace routing and board outline. Added mounting holes.
Parts:
- S1, S2, S3, S4, S5: symbol Logic_74xx:DPDT-Button -> Timer-rescue:DPDT-Button-Logic_74xx
- U2: symbol PiKwonDo:74HC165_PKD -> Timer-rescue:74HC165_PKD-PiKwonDo
Changed lines of the file:
@@
 $EndComp
 $Comp
-L Logic_74xx:DPDT-Button S5
+L Timer-rescue:DPDT-Button-Logic_74xx S5
 U 1 1 5B2D9B30
 P 9850 5700
@@
 $EndComp
 $Comp
-L Logic_74xx:DPDT-Button S1
+L Timer-rescue:DPDT-Button-Logic_74xx S1
 U 1 1 5B2D9E5E
 P 9850 2100
@@
 $EndComp
 $Comp
-L Logic_74xx:DPDT-Button S2
+L Timer-rescue:DPDT-Button-Logic_74xx S2
 U 1 1 5B2D9EA4
 P 9850 3000
@@
 $EndComp
 $Comp
-L Logic_74xx:DPDT-Button S3
+L Timer-rescue:DPDT-Button-Logic_74xx S3
 U 1 1 5B2D9EFB
 P 9850 3900
@@
 $EndComp
 $Comp
-L Logic_74xx:DPDT-Button S4
+L Timer-rescue:DPDT-Button-Logic_74xx S4
 U 1 1 5B2D9F4B
 P 9850 4800
@@
 $EndComp
 $Comp
-L PiKwonDo:74HC165_PKD U2
+L Timer-rescue:74HC165_PKD-PiKwonDo U2
 U 1 1 5B5E202F
 P 7700 2200
@@
 $EndComp
 $Comp
-L power:GND #PWR017
-U 1 1 5B5E67F9
-P 8300 2750
-F 0 "#PWR017" H 8300 2500 50  0001 C CNN
-F 1 "GND" H 8300 2600 50  0000 C CNN
-F 2 "" H 8300 2750 50  0001 C CNN
-F 3 "" H 8300 2750 50  0001 C CNN
-	1    8300 2750
-	0    -1   1    0
-$EndComp
-$Comp
 L power:GND #PWR018
 U 1 1 5B5E6846
@@
 	9000 2150 8300 2150
 Wire Wire Line
-	8900 1300 8900 2300
-Wire Wire Line
-	8900 2300 8300 2300
-Wire Wire Line
 	8800 2900 8800 5450
 Wire Wire Line
 	9200 1300 9200 1850
-Wire Wire Line
-	8300 2900 8800 2900
-Connection ~ 8800 2900
 Wire Wire Line
 	2000 3300 2900 3300
@@
 Connection ~ 9100 2000
 Connection ~ 9000 2150
-Connection ~ 8900 2300
 Connection ~ 9200 1850
 Wire Wire Line
@@
 Wire Wire Line
 	9000 2150 9000 3650
-Wire Wire Line
-	8900 2300 8900 4550
 Wire Wire Line
 	9200 1850 9300 1850
@@
 	1    0    0    -1
 $EndComp
+Wire Wire Line
+	8900 2300 8900 4550
+Wire Wire Line
+	8900 1300 8900 2300
+Connection ~ 8900 2300
+Wire Wire Line
+	8900 2300 8300 2300
+Connection ~ 8800 2900
+Wire Wire Line
+	8300 2900 8800 2900
+$Comp
+L power:GND #PWR017
+U 1 1 5B5E67F9
+P 8300 2750
+F 0 "#PWR017" H 8300 2500 50  0001 C CNN
+F 1 "GND" H 8300 2600 50  0000 C CNN
+F 2 "" H 8300 2750 50  0001 C CNN
+F 3 "" H 8300 2750 50  0001 C CNN
+	1    8300 2750
+	0    -1   1    0
+$EndComp
 $EndSCHEMATC
