File: Electronics/Judge/JudgeBoard.sch (KiCad schematic (older format))
At the start: 28 parts, among them J1 RJ12-UNSHLD, U1 74HC165, U2 74HC165

Commit message: Updated footprints
Parts:
- removed D3, D4, D5: D_Zener, symbol D_Zener
- added D3: D_Zener_Quad, TO_SOT_Packages_SMD:SOT-553, symbol D_Zener_Quad
- C1, C2, C4: footprint Capacitors_THT:C_Disc_D3.4mm_W2.1mm_P2.50mm -> Capacitors_SMD:C_0603_HandSoldering
- C3: footprint Capacitors_THT:CP_Axial_L11.0mm_D5.0mm_P18.00mm_Horizontal -> Capacitors_SMD:C_1210_HandSoldering
- D2: footprint (none) -> Diodes_SMD:D_SMA_Handsoldering
- R1, R2, R3, R4: footprint Resistors_THT:R_Axial_DIN0207_L6.3mm_D2.5mm_P2.54mm_Vertical -> Resistors_SMD:R_1206_HandSoldering
Connections:
- wire segments 75 -> 72
- no-connect marks 38 -> 39
Changed lines of the file:
@@
 LIBS:Logic_CMOS_IEEE
 LIBS:Switch
+LIBS:PiKwonDo
 LIBS:JudgeBoard-cache
 EELAYER 25 0
@@
 	9100 4800 8250 4800
 Wire Wire Line
+	8750 2250 9200 2250
+Wire Wire Line
 	9100 2250 9100 4800
 $Comp
@@
 F 0 "C1" H 7325 1500 50  0000 L CNN
 F 1 "270pF" H 7325 1300 50  0000 L CNN
-F 2 "Capacitors_THT:C_Disc_D3.4mm_W2.1mm_P2.50mm" H 7338 1250 50  0001 C CNN
+F 2 "Capacitors_SMD:C_0603_HandSoldering" H 7338 1250 50  0001 C CNN
 F 3 "" H 7300 1400 50  0001 C CNN
 	1    7300 1400
@@
 F 0 "C2" H 8275 3900 50  0000 L CNN
 F 1 "270pF" H 8275 3700 50  0000 L CNN
-F 2 "Capacitors_THT:C_Disc_D3.4mm_W2.1mm_P2.50mm" H 8288 3650 50  0001 C CNN
+F 2 "Capacitors_SMD:C_0603_HandSoldering" H 8288 3650 50  0001 C CNN
 F 3 "" H 8250 3800 50  0001 C CNN
 	1    8250 3800
@@
 F 0 "C3" H 7675 2500 50  0000 L CNN
 F 1 "10uF" H 7675 2300 50  0000 L CNN
-F 2 "Capacitors_THT:CP_Axial_L11.0mm_D5.0mm_P18.00mm_Horizontal" H 7650 2400 50  0001 C CNN
+F 2 "Capacitors_SMD:C_1210_HandSoldering" H 7650 2400 50  0001 C CNN
 F 3 "" H 7650 2400 50  0001 C CNN
 	1    7650 2400
@@
 F 0 "R1" V 10030 1850 50  0000 C CNN
 F 1 "68" V 9950 1850 50  0000 C CNN
-F 2 "Resistors_THT:R_Axial_DIN0207_L6.3mm_D2.5mm_P2.54mm_Vertical" V 9880 1850 50  0001 C CNN
+F 2 "Resistors_SMD:R_1206_HandSoldering" V 9880 1850 50  0001 C CNN
 F 3 "" H 9950 1850 50  0001 C CNN
 	1    9950 1850
@@
 L GND #PWR026
 U 1 1 5B2837C7
-P 8650 3200
-F 0 "#PWR026" H 8650 2950 50  0001 C CNN
-F 1 "GND" H 8650 3050 50  0000 C CNN
-F 2 "" H 8650 3200 50  0001 C CNN
-F 3 "" H 8650 3200 50  0001 C CNN
-	1    8650 3200
+P 8650 3500
+F 0 "#PWR026" H 8650 3250 50  0001 C CNN
+F 1 "GND" H 8650 3350 50  0000 C CNN
+F 2 "" H 8650 3500 50  0001 C CNN
+F 3 "" H 8650 3500 50  0001 C CNN
+	1    8650 3500
 	1    0    0    -1
 $EndComp
@@
 NoConn ~ 10200 2450
 NoConn ~ 10200 1950
-$Comp
-L D_Zener D3
-U 1 1 5B42DD94
-P 8300 2900
-F 0 "D3" H 8300 3000 50  0000 C CNN
-F 1 "D_Zener" H 8300 2800 50  0000 C CNN
-F 2 "" H 8300 2900 50  0001 C CNN
-F 3 "" H 8300 2900 50  0001 C CNN
-	1    8300 2900
-	0    1    1    0
-$EndComp
-$Comp
-L D_Zener D5
-U 1 1 5B42DE60
-P 8650 2900
-F 0 "D5" H 8650 3000 50  0000 C CNN
-F 1 "D_Zener" H 8650 2800 50  0000 C CNN
-F 2 "" H 8650 2900 50  0001 C CNN
-F 3 "" H 8650 2900 50  0001 C CNN
-	1    8650 2900
-	0    1    1    0
-$EndComp
-Wire Wire Line
-	8300 3050 8300 3100
 Connection ~ 9900 2150
-$Comp
-L D_Zener D4
-U 1 1 5B42E280
-P 8950 2900
-F 0 "D4" H 8950 3000 50  0000 C CNN
-F 1 "D_Zener" H 8950 2800 50  0000 C CNN
-F 2 "" H 8950 2900 50  0001 C CNN
-F 3 "" H 8950 2900 50  0001 C CNN
-	1    8950 2900
-	0    1    1    0
-$EndComp
 $Comp
 L R R4
@@
 F 0 "R4" V 9830 2050 50  0000 C CNN
 F 1 "10" V 9750 2050 50  0000 C CNN
-F 2 "Resistors_THT:R_Axial_DIN0207_L6.3mm_D2.5mm_P2.54mm_Vertical" V 9680 2050 50  0001 C CNN
+F 2 "Resistors_SMD:R_1206_HandSoldering" V 9680 2050 50  0001 C CNN
 F 3 "" H 9750 2050 50  0001 C CNN
 	1    9750 2050
@@
 	9950 1550 9950 1700
 Wire Wire Line
-	8300 2750 8300 2050
+	8300 2350 8300 2050
 Connection ~ 8300 2050
 Connection ~ 9950 2050
@@
 F 0 "R2" V 9630 2150 50  0000 C CNN
 F 1 "470" V 9550 2150 50  0000 C CNN
-F 2 "Resistors_THT:R_Axial_DIN0207_L6.3mm_D2.5mm_P2.54mm_Vertical" V 9480 2150 50  0001 C CNN
+F 2 "Resistors_SMD:R_1206_HandSoldering" V 9480 2150 50  0001 C CNN
 F 3 "" H 9550 2150 50  0001 C CNN
 	1    9550 2150
@@
 F 0 "R3" V 9430 2250 50  0000 C CNN
 F 1 "470" V 9350 2250 50  0000 C CNN
-F 2 "Resistors_THT:R_Axial_DIN0207_L6.3mm_D2.5mm_P2.54mm_Vertical" V 9280 2250 50  0001 C CNN
+F 2 "Resistors_SMD:R_1206_HandSoldering" V 9280 2250 50  0001 C CNN
 F 3 "" H 9350 2250 50  0001 C CNN
 	1    9350 2250
@@
 F 0 "C4" H 9675 2600 50  0000 L CNN
 F 1 "270pF" H 9675 2400 50  0000 L CNN
-F 2 "Capacitors_THT:C_Disc_D3.4mm_W2.1mm_P2.50mm" H 9688 2350 50  0001 C CNN
+F 2 "Capacitors_SMD:C_0603_HandSoldering" H 9688 2350 50  0001 C CNN
 F 3 "" H 9650 2500 50  0001 C CNN
 	1    9650 2500
@@
 F 0 "D2" H 8000 2150 50  0000 C CNN
 F 1 "D_Schottky" H 8000 1950 50  0000 C CNN
-F 2 "" H 8000 2050 50  0001 C CNN
+F 2 "Diodes_SMD:D_SMA_Handsoldering" H 8000 2050 50  0001 C CNN
 F 3 "" H 8000 2050 50  0001 C CNN
 	1    8000 2050
@@
 	8150 2050 9600 2050
 Wire Wire Line
-	8300 3100 8950 3100
-Wire Wire Line
-	8650 3050 8650 3200
-Connection ~ 8650 3100
-Wire Wire Line
-	8950 3100 8950 3050
-Wire Wire Line
-	8650 2750 8650 2150
+	8650 2150 8650 2400
 Connection ~ 8650 2150
-Wire Wire Line
-	9100 2250 9200 2250
-Wire Wire Line
-	8950 2750 8950 2600
-Wire Wire Line
-	8950 2600 9100 2600
-Connection ~ 9100 2600
+Connection ~ 9100 2250
+$Comp
+L D_Zener_Quad D3
+U 1 1 5B443D17
+P 8650 2950
+F 0 "D3" H 8850 3100 60  0000 C CNN
+F 1 "D_Zener_Quad" H 8650 3250 60  0000 C CNN
+F 2 "TO_SOT_Packages_SMD:SOT-553" H 8200 3400 60  0001 C CNN
+F 3 "" H 8200 3400 60  0001 C CNN
+	1    8650 2950
+	0    1    1    0
+$EndComp
+Wire Wire Line
+	8300 2350 8550 2350
+Wire Wire Line
+	8550 2350 8550 2400
+Wire Wire Line
+	8750 2250 8750 2400
+NoConn ~ 8850 2400
 $EndSCHEMATC

Commit message: Updated Judge PCB layout to include new footprints
Parts:
- removed D3: D_Zener_Quad, TO_SOT_Packages_SMD:SOT-553, symbol D_Zener_Quad
- added D3, D4, D5: D_Zener, Diodes_SMD:SOD-80C, symbol D_Zener
Connections:
- wire segments 72 -> 75
- no-connect marks 39 -> 38
Changed lines of the file:
@@
 LIBS:Logic_CMOS_4000
 LIBS:Logic_CMOS_IEEE
+LIBS:PiKwonDo
 LIBS:Switch
-LIBS:PiKwonDo
 LIBS:JudgeBoard-cache
 EELAYER 25 0
@@
 	9100 4800 8250 4800
 Wire Wire Line
-	8750 2250 9200 2250
+	8950 2250 9200 2250
 Wire Wire Line
 	9100 2250 9100 4800
@@
 	9950 1550 9950 1700
 Wire Wire Line
-	8300 2350 8300 2050
+	8300 2050 8300 2750
 Connection ~ 8300 2050
 Connection ~ 9950 2050
@@
 Wire Wire Line
 	8150 2050 9600 2050
-Wire Wire Line
-	8650 2150 8650 2400
+Connection ~ 9100 2250
+$Comp
+L D_Zener D3
+U 1 1 5B4577C8
+P 8350 2900
+F 0 "D3" H 8350 3000 50  0000 C CNN
+F 1 "D_Zener" H 8350 2800 50  0000 C CNN
+F 2 "Diodes_SMD:SOD-80C" H 8350 2900 50  0001 C CNN
+F 3 "" H 8350 2900 50  0001 C CNN
+	1    8350 2900
+	0    1    1    0
+$EndComp
+$Comp
+L D_Zener D4
+U 1 1 5B457892
+P 8650 2900
+F 0 "D4" H 8650 3000 50  0000 C CNN
+F 1 "D_Zener" H 8650 2800 50  0000 C CNN
+F 2 "Diodes_SMD:SOD-80C" H 8650 2900 50  0001 C CNN
+F 3 "" H 8650 2900 50  0001 C CNN
+	1    8650 2900
+	0    1    1    0
+$EndComp
+$Comp
+L D_Zener D5
+U 1 1 5B4578F4
+P 8950 2900
+F 0 "D5" H 8950 3000 50  0000 C CNN
+F 1 "D_Zener" H 8950 2800 50  0000 C CNN
+F 2 "Diodes_SMD:SOD-80C" H 8950 2900 50  0001 C CNN
+F 3 "" H 8950 2900 50  0001 C CNN
+	1    8950 2900
+	0    1    1    0
+$EndComp
+Wire Wire Line
+	8300 2750 8350 2750
+Wire Wire Line
+	8650 2750 8650 2150
 Connection ~ 8650 2150
-Connection ~ 9100 2250
-$Comp
-L D_Zener_Quad D3
-U 1 1 5B443D17
-P 8650 2950
-F 0 "D3" H 8850 3100 60  0000 C CNN
-F 1 "D_Zener_Quad" H 8650 3250 60  0000 C CNN
-F 2 "TO_SOT_Packages_SMD:SOT-553" H 8200 3400 60  0001 C CNN
-F 3 "" H 8200 3400 60  0001 C CNN
-	1    8650 2950
-	0    1    1    0
-$EndComp
-Wire Wire Line
-	8300 2350 8550 2350
-Wire Wire Line
-	8550 2350 8550 2400
-Wire Wire Line
-	8750 2250 8750 2400
-NoConn ~ 8850 2400
+Wire Wire Line
+	8950 2750 8950 2250
+Wire Wire Line
+	8350 3050 8350 3350
+Wire Wire Line
+	8350 3350 8950 3350
+Wire Wire Line
+	8650 3050 8650 3500
+Connection ~ 8650 3350
+Wire Wire Line
+	8950 3350 8950 3050
 $EndSCHEMATC

Commit message: Updated Judge PCB for manufacturability
Parts:
- C1, C2, C4: symbol C -> device:C
- C3: symbol CP1 -> device:CP1
- D1: symbol LED -> device:LED
- D2: symbol D_Schottky -> device:D_Schottky
- D3, D4, D5: symbol D_Zener -> device:D_Zener
- J1: symbol RJ12-UNSHLD -> PiKwonDo:RJ12-UNSHLD
- R1, R2, R3, R4: symbol R -> device:R
- RN1, RN2: symbol R_Network05 -> device:R_Network05
- S1, S10, S2, S3, S5, S7, S8, S9: symbol DPDT-Button -> PiKwonDo:DPDT-Button
- S4, S6: symbol DPST-Button -> JudgeBoard-rescue:DPST-Button
- U1, U2: symbol 74HC165 -> JudgeBoard-rescue:74HC165
Connections:
- wire segments 75 -> 95

Commit message: Updating judge circuits and pcb to match timer
Parts:
- removed C3: 10uF, Capacitors_SMD:C_1210_HandSoldering, symbol device:CP1
- removed D4: D_Zener, Diodes_SMD:SOD-80C, symbol device:D_Zener
- added C3: 1uF, Capacitor_SMD:C_1206_3216Metric_Pad1.42x1.75mm_HandSolder, symbol device:C
- added R5: 470, Resistor_SMD:R_1206_3216Metric_Pad1.42x1.75mm_HandSolder, symbol device:R
- added U3: MIC5504-3.3YM5, Package_TO_SOT_SMD:SOT-23-5, symbol Regulator_Linear:MIC5504-3.3YM5
- C1, C2: value 270pF -> 1uF; footprint Capacitors_SMD:C_0603_HandSoldering -> Capacitor_SMD:C_1206_3216Metric_Pad1.42x1.75mm_HandSolder
- C4: value 270pF -> 470pF; footprint Capacitors_SMD:C_0603_HandSoldering -> Capacitor_SMD:C_1206_3216Metric_Pad1.42x1.75mm_HandSolder
- D1: footprint LEDs:LED_D2.0mm_W4.8mm_H2.5mm_FlatTop -> LED_THT:LED_D3.0mm_Spread
- D3: value D_Zener -> 3.3V; footprint Diodes_SMD:SOD-80C -> Diode_SMD:D_1206_3216Metric_Pad1.42x1.75mm_HandSolder
- D5: value D_Zener -> 5V
- R1: value 68 -> 470; footprint Resistors_SMD:R_1206_HandSoldering -> Resistor_SMD:R_1206_3216Metric_Pad1.42x1.75mm_HandSolder
- R2: value 470 -> 10; footprint Resistors_SMD:R_1206_HandSoldering -> Resistor_SMD:R_1206_3216Metric_Pad1.42x1.75mm_HandSolder
- R3: footprint Resistors_SMD:R_1206_HandSoldering -> Resistor_SMD:R_1206_3216Metric_Pad1.42x1.75mm_HandSolder
- R4: value 10 -> 100; footprint Resistors_SMD:R_1206_HandSoldering -> Resistor_SMD:R_1206_3216Metric_Pad1.42x1.75mm_HandSolder
- RN1, RN2: footprint Resistors_THT:R_Array_SIP6 -> Resistor_THT:R_Array_SIP6
- U1, U2: symbol JudgeBoard-rescue:74HC165 -> PiKwonDo:74HC165
Connections:
- net labels added: +5V, Q, Q_intermediate
- wire segments 95 -> 88
- no-connect marks 38 -> 14
Other:
- moved on the sheet: S4, S6, U1, U2

Commit message: Intermediate commit while moving components to final locations.
Parts:
- removed J1: RJ12-UNSHLD, PiKwonDo:TH-RJ12, symbol PiKwonDo:RJ12-UNSHLD
- added C5, C6: 470pF, Capacitor_SMD:C_1206_3216Metric_Pad1.42x1.75mm_HandSolder, symbol device:C
- added J1: RJ10, Local_lib:RJ14, symbol Connector:RJ10
Connections:
- net labels added: Q_inter
- net labels removed: Q_intermediate
- wire segments 88 -> 89
- no-connect marks 14 -> 12
Other:
- moved on the sheet: S4, U3

Commit message: Finalized trace routing and part placement.
Parts:
- C1, C2, C3, C4, C5, C6: symbol device:C -> JudgeBoard-rescue:C-device
- D1: symbol device:LED -> JudgeBoard-rescue:LED-device
- D2: symbol device:D_Schottky -> JudgeBoard-rescue:D_Schottky-device
- D3, D5: symbol device:D_Zener -> JudgeBoard-rescue:D_Zener-device
- R1, R2, R3, R4, R5: symbol device:R -> JudgeBoard-rescue:R-device
- RN1, RN2: symbol device:R_Network05 -> JudgeBoard-rescue:R_Network05-device
- S1, S10, S2, S3, S5, S7, S8, S9: symbol PiKwonDo:DPDT-Button -> JudgeBoard-rescue:DPDT-Button-PiKwonDo
- U1, U2: symbol PiKwonDo:74HC165 -> JudgeBoard-rescue:74HC165-PiKwonDo
Other:
- moved on the sheet: U1, U2

Commit message: Updated boards for two-sided manufacture.
Parts:
- J1: symbol Connector:RJ10 -> JudgeBoard-rescue:RJ10-Connector
- U3: symbol Regulator_Linear:MIC5504-3.3YM5 -> JudgeBoard-rescue:MIC5504-3.3YM5-Regulator_Linear
Changed lines of the file:
@@
 EESchema Schematic File Version 4
 LIBS:JudgeBoard-cache
-EELAYER 26 0
+EELAYER 30 0
 EELAYER END
 $Descr A4 11693 8268
@@
 $EndComp
 $Comp
-L power:+5V #PWR0102
+L JudgeBoard-rescue:+5V-power #PWR0102
 U 1 1 5BDE9457
 P 1450 800
@@
 $EndComp
 $Comp
-L power:+5V #PWR0103
+L JudgeBoard-rescue:+5V-power #PWR0103
 U 1 1 5BDE9534
 P 3800 2050
@@
 $EndComp
 $Comp
-L Regulator_Linear:MIC5504-3.3YM5 U3
+L JudgeBoard-rescue:MIC5504-3.3YM5-Regulator_Linear U3
 U 1 1 5BDFC1D2
 P 4150 2600
@@
 $EndComp
 $Comp
-L Connector:RJ10 J1
+L JudgeBoard-rescue:RJ10-Connector J1
 U 1 1 5C3EA0C7
 P 900 2250
