File: Electronics/Judge/JudgeBoard.kicad_pcb (KiCad board)
At the start: 2 copper layers, 119 x 53 mm, 33 parts, among them J1 RJ10, M3 MountingHole_3.2mm_M3, U1 74HC165, U2 74HC165, U3 MIC5504-3.3YM5

Commit message: Updated component sourcing
Routing:
- net +3V3: track 142.9 -> 134.5 mm
